File: Eagle/CrackberryPi.brd (EAGLE design)
At the start: 100 x 80 mm, 23 parts, among them IC1 X1205IS8, IC2 24C02CSM, J1 22-27-2031-03, Q1 MC-406, X1 1503_07, X2 057-040-1

Commit message: scherm en touchscreen bestanden en info
Parts:
- removed SJ1, SJ2: (no value), jumper:SJ
- added C6, C7: (no value), rcl:C0603
- added R7: 10k, rcl:R0603
- added TP1_WP, TP2_WP: TPSTP15R, testpad:TP15R
- added U$3: ADS7843, ads7843:SOP16
- added WP_GND: (no value), jumper:SJ
- added X3: FH28-50S-0.5SH(51), con-hirose:FH28-50S-0.5SH(51)
- moved R6 158.8 mm to (73.9, 75.9)
- moved R5 150.5 mm to (70.5, 74.3)
- moved C5 150.2 mm to (71.2, 67.8)
- moved R4 146.6 mm to (70.7, 71.4)
- moved IC2 145.4 mm to (76.8, 69.8)
- moved J1 46.7 mm to (49.6, 71.7), turned to 90 degrees
- moved X1 29.6 mm to (49.4, 74.2)
- moved G1 21.0 mm to (10.9, 13.7)
Connections:
- removed net N$12: R6.2, SJ2.1
- new net INTERRUPT: R7.1, U$3.11
- new net TOUCH_X+: U$3.2
- new net TOUCH_X-: U$3.4
- new net TOUCH_Y+: U$3.3
- new net TOUCH_Y-: U$3.5
- net +3V3: now also C6.1, C7.1, R6.2, R7.2, U$3.1, U$3.10, U$3.9; no longer SJ2.2
- net GND: now also C6.2, C7.2, TP1_WP.TP, U$3.6, WP_GND.1; no longer SJ1.1
- net N$11: now also TP2_WP.TP, WP_GND.2; no longer SJ1.2

Commit message: screen info
Parts:
- added C8, C9: (no value), rcl:C0603
- added LED1, LED2, LED3: (no value), eagle-ltspice:LED_SML0603
- added Q2: FDN360P, transistor-power:SUPER-SOT3
- added R10: 1k, rcl:R0603
- added R11, R8, R9: 470, rcl:R0603
- added R12: THERMISTOR-5, varistor:R-5
- added R13, R14, R15, R16, R17, R24: 10k, rcl:R0603
- added R18, R19, R20, R21, R22, R23: 147, rcl:R0603
- added R25: 45k, rcl:R0603
- added SV1: (no value), con-amp-mt:S02P
- added U$4: MCP73833, mcp73833:MSOP10
- added X4: MINI-USB-32005-301, con-cypressindustries:32005-301
Connections:
- new net DE: R17.2
- new net H_SYNC: R15.1
- new net LEDK1: R18.2
- new net LEDK2: R19.2
- new net LEDK3: R20.2
- new net LEDK4: R21.2
- new net LEDK5: R22.2
- new net LEDK6: R23.2
- new net LED_ON: R24.2, R25.2
- new net N$12: Q2.2, R18.1, R19.1, R20.1, R21.1, R22.1, R23.1
- new net N$13: R8.2, U$4.3
- new net N$14: LED1.C, R8.1
- new net N$15: R9.2, U$4.4
- new net N$16: R11.2, U$4.7
- new net N$17: LED3.C, R11.1
- new net N$18: LED2.C, R9.1
- new net N$19: R10.2, U$4.6
- new net N$20: Q2.1, R24.1
- new net N$21: R12.1, U$4.8
- new net N$22: C8.1, SV1.2, U$4.10, U$4.9
- new net P_CLK: R16.2
- new net RST: R13.1
- new net V+: LED1.A, LED2.A, LED3.A, U$4.1, U$4.2, X4.1
- new net V_SYNC: R14.1
- net +3V3: now also R13.2, R14.2, R15.2, X3.2, X3.3, X3.4, X3.5
- net +5V: now also C9.1
- net GND: now also C8.2, C9.2, Q2.3, R10.1, R12.2, R16.1, R17.1, R25.1, SV1.1, U$4.5, X3.1, X3.14, X3.15, X3.16, X3.17, X3.18, X3.19, X3.20, X3.21, X3.22, X3.23, X3.24, X3.25, X3.26, X3.27, X3.28, X3.29, X3.30, X3.31, X3.32, X3.6, X3.7, X3.8, X4.5

Commit message: part selection
Parts:
- removed G1: CR2430H, battery:CR2430H
- removed IC1: X1205IS8, xicor:SO-08
- removed J1: 22-27-2031-03, con-molex:6410-03
- removed Q1: MC-406, crystal:MC-406
- removed TP1_WP, TP2_WP: TPSTP15R, testpad:TP15R
- removed X1: 1503_07, con-lumberg:1503_07
- added Q3: (no value), crystal:MM20SS
- added R26: PC16SV, piher:PC16SV
- added U$5: MCP7940N, MCP7940N:SO08
- added U$6: CR2032, cr2032:CR2032
- added WP_GND1: (no value), jumper:SJ
- moved U$3 109.0 mm to (33.0, -95.6)
- moved C6 97.7 mm to (26.9, -86.7)
- moved R7 94.9 mm to (33.4, -82.3)
- moved C7 94.5 mm to (24.1, -84.2)
- moved R5 72.4 mm to (38.8, 9.20), flipped to the bottom
- moved R6 71.2 mm to (39.3, 13.7), flipped to the bottom, turned to 90 degrees
- moved R4 68.1 mm to (38.8, 11.2), flipped to the bottom
- moved WP_GND 68.0 mm to (46.4, 16.8), flipped to the bottom
- moved R1 67.5 mm to (72.5, 17.5), flipped to the bottom
- moved C5 65.7 mm to (36.1, 12.3), flipped to the bottom, turned to 90 degrees
- moved IC2 65.6 mm to (46.3, 11.7), flipped to the bottom, turned to 270 degrees
- moved R3 64.9 mm to (72.5, 20.3), flipped to the bottom
- moved C1 56.2 mm to (68.9, 17.0), flipped to the bottom, turned to 270 degrees
- moved X3 53.8 mm to (6.50, 40.4), flipped to the bottom, turned to 90 degrees
- moved X2 52.4 mm to (52.4, 3.30), turned to 180 degrees
Connections:
- net GPIO14 renamed UART_TX
- net GPIO15 renamed UART_RX
- removed net GPIO10: X2.19
- removed net GPIO17: X2.11
- removed net GPIO4: X2.7
- removed net GPIO9: X2.21
- removed net LED_ON: R24.2, R25.2
- removed net N$4: J1.1, X1.2@1
- removed net N$5: J1.2, X1.3
- removed net N$6: J1.3, X1.1
- new net ADDITIONAL_1: U$3.7
- new net ADDITIONAL_2: U$3.8
- new net MISO: X2.21
- new net MOSI: X2.19
- new net N$23: R26.1A, R26.S2
- new net N$25: R26.1S
- new net PWM: R24.2, R25.2, X2.11
- net +3V3: now also U$5.8; no longer IC1.8
- net +5V: now also R26.S1
- net GND: now also R26.1E, U$5.4, U$6.GND, WP_GND1.1; no longer G1.-, IC1.4, TP1_WP.TP
- net INT: now also U$5.7, X2.7; no longer IC1.3
- net N$1: now also Q3.1, U$5.2; no longer IC1.1, Q1.4
- net N$11: no longer TP2_WP.TP
- net N$12: now also WP_GND1.2
- net N$2: now also Q3.4, U$5.1; no longer IC1.2, Q1.1
- net N$3: now also U$5.3, U$6.+; no longer G1.+, IC1.7
- net SCL_3V3: now also U$5.6; no longer IC1.6
- net SDA_3V3: now also U$5.5; no longer IC1.5
Routing:
- net +3V3: track 0.00 -> 21.9 mm
- net SDA_3V3: track 0.00 -> 18.7 mm
- net N$3: track 0.00 -> 17.8 mm
- net SCL_3V3: track 0.00 -> 17.3 mm
- net ID_SC: track 0.00 -> 14.4 mm
- net INT: track 0.00 -> 13.2 mm
- net N$11: track 0.00 -> 10.7 mm
- net ID_SD: track 0.00 -> 9.03 mm
- net N$1: track 0.00 -> 8.02 mm
- net N$2: track 0.00 -> 6.58 mm
- net +5V: track 0.00 -> 2.54 mm
- added copper zone on layer 1, net GND
- added copper zone on layer 16, net GND
Other:
- board size 100 x 80 mm -> 85 x 86 mm

Commit message: pcb
Parts:
- moved X3 21.6 mm to (25.2, 29.6)
Changed lines of the file:
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@@
 <element name="C6" library="rcl" package="C0603" value="" x="26.9" y="-86.7"/>
 <element name="C7" library="rcl" package="C0603" value="" x="24.1" y="-84.2"/>
-<element name="X3" library="con-hirose" package="FH28-50S-0.5SH(51)" value="FH28-50S-0.5SH(51)" x="6.5" y="40.4" rot="MR90">
-<attribute name="OC_NEWARK" value="unknown" x="6.5" y="40.4" size="1.778" layer="28" rot="MR90" display="off"/>
-<attribute name="MPN" value="" x="6.5" y="40.4" size="1.778" layer="28" rot="MR90" display="off"/>
-<attribute name="MF" value="" x="6.5" y="40.4" size="1.778" layer="28" rot="MR90" display="off"/>
-<attribute name="OC_FARNELL" value="unknown" x="6.5" y="40.4" size="1.778" layer="28" rot="MR90" display="off"/>
+<element name="X3" library="con-hirose" package="FH28-50S-0.5SH(51)" value="FH28-50S-0.5SH(51)" x="25.2" y="29.6" rot="MR90">
+<attribute name="OC_NEWARK" value="unknown" x="25.2" y="29.6" size="1.778" layer="28" rot="MR90" display="off"/>
+<attribute name="MPN" value="" x="25.2" y="29.6" size="1.778" layer="28" rot="MR90" display="off"/>
+<attribute name="MF" value="" x="25.2" y="29.6" size="1.778" layer="28" rot="MR90" display="off"/>
+<attribute name="OC_FARNELL" value="unknown" x="25.2" y="29.6" size="1.778" layer="28" rot="MR90" display="off"/>
 </element>
 <element name="U$4" library="mcp73833" package="MSOP10" value="MCP73833" x="-5.3" y="-15.2"/>
@@
 <wire x1="-6.65" y1="-57.5" x2="-2.86" y2="-52.3" width="0" layer="19" extent="1-1"/>
 <wire x1="1.8" y1="-28.2" x2="-8.35" y2="-47.1" width="0" layer="19" extent="1-1"/>
-<wire x1="10" y1="30.65" x2="10" y2="28.15" width="0" layer="19" extent="16-16"/>
-<wire x1="10" y1="34.65" x2="10" y2="31.65" width="0" layer="19" extent="16-16"/>
+<wire x1="28.7" y1="19.85" x2="28.7" y2="17.35" width="0" layer="19" extent="16-16"/>
+<wire x1="28.7" y1="23.85" x2="28.7" y2="20.85" width="0" layer="19" extent="16-16"/>
 <wire x1="-4.3" y1="-17.3131" x2="1.8" y2="-28.2" width="0" layer="19" extent="1-1"/>
 <wire x1="12.38" y1="66.21" x2="4.5" y2="52" width="0" layer="19" extent="1-1"/>
@@
 <wire x1="56.24" y1="4.57" x2="34.25" y2="-82.3" width="0" layer="19" extent="1-1"/>
 <wire x1="42.97" y1="13.605" x2="56.24" y2="4.57" width="0" layer="19" extent="16-16"/>
+<wire x1="28.7" y1="17.85" x2="36.1" y2="11.45" width="0" layer="19" extent="16-16"/>
+<wire x1="28.7" y1="18.35" x2="28.7" y2="17.85" width="0" layer="19" extent="16-16"/>
+<wire x1="28.7" y1="18.85" x2="28.7" y2="18.35" width="0" layer="19" extent="16-16"/>
+<wire x1="28.7" y1="19.35" x2="28.7" y2="18.85" width="0" layer="19" extent="16-16"/>
 <wire x1="68.86" y1="17.85" x2="56.24" y2="4.57" width="0" layer="19" extent="16-16"/>
 <wire x1="76.56" y1="4.57" x2="74.1" y2="15.505" width="0" layer="19" extent="16-16"/>
-<wire x1="10" y1="28.65" x2="36.1" y2="11.45" width="0" layer="19" extent="16-16"/>
-<wire x1="10" y1="29.15" x2="10" y2="28.65" width="0" layer="19" extent="16-16"/>
-<wire x1="10" y1="29.65" x2="10" y2="29.15" width="0" layer="19" extent="16-16"/>
-<wire x1="10" y1="30.15" x2="10" y2="29.65" width="0" layer="19" extent="16-16"/>
 </signal>
 <signal name="INT">

Commit message: pcb development
Parts:
- removed C6: (no value), rcl:C0603
- removed D1: (no value), diode:SOD80C
- removed SV1: (no value), con-amp-mt:S02P
- removed U$2: MAX2650, MAX2650:SOT143
- removed U$3: ADS7843, ads7843:SOP16
- removed WP_GND, WP_GND1: (no value), jumper:SJ
- removed X3: FH28-50S-0.5SH(51), con-hirose:FH28-50S-0.5SH(51)
- removed X4: MINI-USB-32005-301, con-cypressindustries:32005-301
- added C10: 1mf, rcl:C0603
- added C11: 10nf, rcl:C0603
- added C12, C13, C14, C15: 0.1mf, rcl:C0603
- added C16: 22mf, rcl:C0805
- added C17: 10mf, rcl:C0805
- added C18: (no value), rcl:C0603
- added D2: (no value), diode:SOD80C
- added D3: BAS40-05, diode:SOT23
- added IC1: REG1117, burr-brown:SOT223
- added L2: (no value), rcl:L4532P
- added Q1: (no value), semicon-smd-ipc:SOT23
- added R27: 1k, rcl:R0603
- added R28, R29, R34, R35: 10k, rcl:R0603
- added R30, R32: 2m, rcl:R0603
- added R31, R33: 220k, rcl:R0603
- added S1: (no value), switch:255SB
- added SJ1: (no value), jumper:SJ
- added U$7: MAX17043, MAX17043:DFN-2X3
- added U$8: TPS61200, TPS61200:MCP73833
- added U$9: MICRO_USB, MICRO_USB:MICRO_USB
- added X1: 53261-02, con-molex:53261-02
- added X5: FH12-50S-0.5SH, FCI_62684:FH12-50S-0.5SH
- R12: value THERMISTOR-5 -> 10k; device varistor:R-5 -> rcl:R0603
- R2: value (none) -> THERMISTOR-2,5; device rcl:R0603 -> varistor:RS-2,5
- R26: value PC16SV -> 10k; device piher:PC16SV -> rcl:R0603
- R6: value 1k -> 10k
- U$1: value MAX2650 -> TSC2046; device MAX2650:SOT143 -> tsc2046:TSSOP16
- moved R26 195.1 mm to (28.7, 44.8), flipped to the bottom, turned to 90 degrees
- moved R25 157.2 mm to (47.4, 8.30), flipped to the bottom
- moved R24 154.4 mm to (47.4, 9.80), flipped to the bottom
- moved R23 153.6 mm to (55.9, 16.0), flipped to the bottom
- moved R22 150.7 mm to (55.9, 17.4), flipped to the bottom
- moved Q2 149.4 mm to (50.6, 8.70), flipped to the bottom, turned to 180 degrees
- moved R21 147.9 mm to (55.9, 18.8), flipped to the bottom
- moved R20 145.2 mm to (55.9, 20.2), flipped to the bottom
- moved R19 142.4 mm to (55.9, 21.6), flipped to the bottom
- moved R18 139.7 mm to (55.9, 23.0), flipped to the bottom
- moved C9 138.1 mm to (55.9, 24.4), flipped to the bottom, turned to 180 degrees
- moved R17 135.4 mm to (55.9, 25.8), flipped to the bottom
- moved R16 132.8 mm to (55.9, 27.2), flipped to the bottom
- moved C8 130.8 mm to (70.4, 47.6), flipped to the bottom
- moved R15 130.2 mm to (55.9, 28.6), flipped to the bottom, turned to 180 degrees
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Connections:
- net GPIO7 renamed CE1
- net GPIO8 renamed CE0
- removed net +15V: D1.C
- removed net ADDITIONAL_1: U$3.7
- removed net ADDITIONAL_2: U$3.8
- removed net GPIO11: X2.23
- removed net INTERRUPT: R7.1, U$3.11
- removed net N$10: C3.1, D1.A, R2.2
- removed net N$11: IC2.7, R6.1, WP_GND.2
- removed net N$16: R11.2, U$4.7
- removed net N$25: R26.1S
- removed net N$7: U$1.3, U$2.1
- removed net N$8: C3.2, U$1.1
- removed net N$9: C2.1, U$2.3
- removed net RANDOM_OUTPUT: C2.2
- removed net V+: LED1.A, LED2.A, LED3.A, U$4.1, U$4.2, X4.1
- new net +5V/4: C9.1, X5.43
- new net 2046_BUSY: R34.1, U$1.13
- new net 2046_CS: R6.1, U$1.15
- new net BAT+: C8.1, R27.1, S1.3, U$4.10, U$4.9, X1.1
- new net CS: X5.38
- new net D/C: X5.37
- new net ENABLE_STEPUP: Q1.2, R11.2, R28.1, U$4.7, U$8.6
- new net N$24: L2.2, U$8.3
- new net N$26: C15.1, U$8.1
- new net N$27: R32.1, R33.2, U$8.10
- new net N$28: D2.C, D3.2, LED1.A, LED2.A, LED3.A, U$4.1, U$4.2, U$9.1_+5V
- new net N$4: R26.1, U$8.5
- new net N$5: C10.1, R27.2, U$7.2
- new net N$6: C16.1, D3.1, R32.2, U$8.2
- new net PENIRQ: R7.1, U$1.11
- new net RD: X5.35
- new net SCK: U$1.16, X2.23, X5.36
- new net VBAT: C12.1, C17.1, L2.1, R26.2, R28.2, R29.2, R30.2, S1.2
- new net VCC: C14.1, C2.1, C3.1, C7.1, IC1.2, R12.2, R13.2, R14.2, R15.2, R34.2, R35.2, R6.2, U$1.1, U$1.10, U$1.9, X5.2, X5.3, X5.4, X5.5
- net +3V3: now also C11.1, U$7.3; no longer C6.1, C7.1, R13.2, R14.2, R15.2, R6.2, R7.2, U$3.1, U$3.10, U$3.9, X3.2, X3.3, X3.4, X3.5
- net +5V: now also C13.1, D3.3, IC1.3, Q1.1; no longer C4.1, C9.1, R26.S1, U$1.4, U$2.4
- net DE: now also X5.13
- net GND: now also C10.2, C11.2, C13.2, C14.2, C15.2, C16.2, C17.2, C18.1, C4.1, D2.A, IC1.1, IC2.7, Q1.3, R2.2, R31.1, R33.1, R7.2, SJ1.1, U$1.6, U$1.7, U$1.8, U$7.1, U$7.4, U$7.6, U$7.EXP, U$8.4, U$8.9, U$8.GND, U$9.4_ID, U$9.5_0V, U$9.GND1, U$9.GND2, U$9.GND3, U$9.GND4, U$9.GND5, U$9.P$1, U$9.P$7, X1.2, X5.1, X5.14, X5.15, X5.16, X5.17, X5.18, X5.19, X5.20, X5.21, X5.22, X5.23, X5.24, X5.25, X5.26, X5.27, X5.28, X5.29, X5.30, X5.31, X5.32, X5.50, X5.6, X5.7, X5.8; no longer C4.2, C6.2, R12.2, R2.1, R26.1E, SV1.1, U$1.2, U$2.2, U$3.6, WP_GND.1, WP_GND1.1, X3.1, X3.14, X3.15, X3.16, X3.17, X3.18, X3.19, X3.20, X3.21, X3.22, X3.23, X3.24, X3.25, X3.26, X3.27, X3.28, X3.29, X3.30, X3.31, X3.32, X3.6, X3.7, X3.8, X4.5
- net H_SYNC: now also X5.11
- net INT: now also U$7.5
- net LEDK1: now also X5.44
- net LEDK2: now also X5.45
- net LEDK3: now also X5.46
- net LEDK4: now also X5.47
- net LEDK5: now also X5.48
- net LEDK6: now also X5.49
- net MISO: now also R35.1, U$1.12, X5.33
- net MOSI: now also R12.1, U$1.14, X5.34
- net N$12: no longer WP_GND1.2
- net N$21: now also R2.1; no longer R12.1
- net N$22: now also R29.1, SJ1.2, U$8.8; no longer C8.1, SV1.2, U$4.10, U$4.9
- net N$23: now also C12.2, R30.1, R31.2, U$8.7; no longer R26.1A, R26.S2
- net P_CLK: now also X5.12
- net RST: now also X5.9
- net SCL_3V3: now also U$7.7
- net SDA_3V3: now also U$7.8
- net TOUCH_X+: now also C2.2, U$1.2, X5.39; no longer U$3.2
- net TOUCH_X-: now also C18.2, U$1.4, X5.41; no longer U$3.4
- net TOUCH_Y+: now also C3.2, U$1.3, X5.42; no longer U$3.3
- net TOUCH_Y-: now also C4.2, U$1.5, X5.40; no longer U$3.5
- net V_SYNC: now also X5.10
Routing:
- net N$21: track 0.00 -> 122.3 mm, vias 0 -> 1
- net BAT+: track 0.00 -> 100.7 mm, vias 0 -> 3
- net +5V: track 2.54 -> 102.1 mm, vias 0 -> 2
- net ENABLE_STEPUP: track 0.00 -> 81.2 mm, vias 0 -> 4
- net N$3: track 17.8 -> 83.8 mm
- net VCC: track 0.00 -> 54.4 mm
- net N$28: track 0.00 -> 52.8 mm
- net +3V3: track 21.9 -> 56.5 mm
- net MOSI: track 0.00 -> 32.3 mm, vias 0 -> 1
- net GND: track 0.00 -> 29.6 mm
- net TOUCH_X+: track 0.00 -> 27.0 mm, vias 0 -> 2
- net MISO: track 0.00 -> 25.7 mm, vias 0 -> 1
- net VBAT: track 0.00 -> 24.2 mm
- net TOUCH_Y-: track 0.00 -> 23.1 mm
- net TOUCH_X-: track 0.00 -> 22.8 mm
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Other:
- outline, holes or cut-outs redrawn
- board text added: "Connector"
- board text added: "HDMI"

Commit message: finalizing pcb first proto
schematics, library parts and gerber rar
Parts:
- removed C10: 1mf, rcl:C0603
- removed C11: 10nf, rcl:C0603
- removed C12, C15: 0.1mf, rcl:C0603
- removed C16: 22mf, rcl:C0805
- removed C17: 10mf, rcl:C0805
- removed D2: (no value), diode:SOD80C
- removed D3: BAS40-05, diode:SOT23
- removed L2: (no value), rcl:L4532P
- removed LED1, LED2, LED3: (no value), eagle-ltspice:LED_SML0603
- removed Q2: FDN360P, transistor-power:SUPER-SOT3
- removed R10, R27: 1k, rcl:R0603
- removed R11, R8, R9: 470, rcl:R0603
- removed R12, R26, R28, R29, R34, R35, R7: 10k, rcl:R0603
- removed R30, R32: 2m, rcl:R0603
- removed R31, R33: 220k, rcl:R0603
- removed S1: (no value), switch:255SB
- removed SJ1: (no value), jumper:SJ
- removed U$1: TSC2046, tsc2046:TSSOP16
- removed U$7: MAX17043, MAX17043:DFN-2X3
- removed U$8: TPS61200, TPS61200:MCP73833
- removed X1: 53261-02, con-molex:53261-02
- added C19: 4.7mf, rcl:C0603
- added C20: 68pf, rcl:C0603
- added C21, C23: 470pf, rcl:C0603
- added C22: 0.1mf, rcl:C0603
- added C6: 10mf, rcl:C0603
- added D1: (no value), diode:SOD123
- added D4: 1N759, diode:SOD80C
- added D5: SFH482, led:SFH482
- added JMP1: 0R-JUMPC, jump-0r-smd:C0R-JMP
- added L1: 8.2mH, rcl:R1210
- added LED4, LED5: (no value), eagle-ltspice:LED_SML0603
- added R36: 1.3m, rcl:R0603
- added R37: 110k, rcl:R0603
- added R38, R39: 30, rcl:R0603
- added R40: 1k, rcl:R0603
- added R41, R42: 10k, rcl:R0603
- added SJ2: (no value), jumper:SJ
- added T1: BC847, transistor:SOT23
- added U$10, U$3: MAX2650, max2650:SOT143-W
- added U$2: NCP1406, ncp1406:SOT23-5L
- added X3: C-GRID-03-70543, con-molex:70543-03
- C13, C14: value 0.1mf -> 4.7mF
- C8: value (none) -> 0.1mf
- C9: value (none) -> 1mf
- Q1: value (none) -> IRLML5203; device semicon-smd-ipc:SOT23 -> transistor-power:MICRO3
- R2: value THERMISTOR-2,5 -> 10k; device varistor:RS-2,5 -> rcl:R0603
- U$4: value MCP73833 -> CR1216; device mcp73833:MSOP10 -> cr1216:CR1216
- U$6: value CR2032 -> TSC2007; device cr2032:CR2032 -> tsc2046:TSSOP16
- moved Q1 50.2 mm to (36.2, 13.5), turned to 180 degrees
- moved C8 41.8 mm to (62.5, 6.60), turned to 270 degrees
- moved U$4 27.3 mm to (56.3, 26.9), turned to 90 degrees
- moved C1 23.3 mm to (50.1, 10.0), turned to 90 degrees
- moved Q3 23.0 mm to (58.9, 12.3)
- moved U$5 21.8 mm to (53.3, 13.3), turned to 180 degrees
- moved R5 20.7 mm to (35.9, 8.90), turned to 90 degrees
- moved C9 20.6 mm to (35.3, 24.3)
- moved R13 20.5 mm to (35.4, 32.4)
- moved R14 20.5 mm to (35.4, 31.0)
- moved R15 20.5 mm to (35.4, 29.6)
- moved R16 20.5 mm to (35.4, 28.2)
- moved R17 20.5 mm to (35.4, 26.8)
- moved R18 20.5 mm to (35.4, 23.0)
- moved R19 20.5 mm to (35.4, 21.6)
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Connections:
- net GPIO21 renamed AVALANCHE_ENABLE
- removed net +5V/4: C9.1, X5.43
- removed net 2046_BUSY: R34.1, U$1.13
- removed net 2046_CS: R6.1, U$1.15
- removed net BAT+: C8.1, R27.1, S1.3, U$4.10, U$4.9, X1.1
- removed net CS: X5.38
- removed net ENABLE_STEPUP: Q1.2, R11.2, R28.1, U$4.7, U$8.6
- removed net GPIO12: X2.32
- removed net GPIO13: X2.33
- removed net GPIO16: X2.36
- removed net GPIO20: X2.38
- removed net GPIO6: X2.31
- removed net N$1: Q3.1, U$5.2
- removed net N$13: R8.2, U$4.3
- removed net N$14: LED1.C, R8.1
- removed net N$15: R9.2, U$4.4
- removed net N$17: LED3.C, R11.1
- removed net N$18: LED2.C, R9.1
- removed net N$19: R10.2, U$4.6
- removed net N$2: Q3.4, U$5.1
- removed net N$21: R2.1, U$4.8
- removed net N$22: R29.1, SJ1.2, U$8.8
- removed net N$23: C12.2, R30.1, R31.2, U$8.7
- removed net N$24: L2.2, U$8.3
- removed net N$26: C15.1, U$8.1
- removed net N$27: R32.1, R33.2, U$8.10
- removed net N$28: D2.C, D3.2, LED1.A, LED2.A, LED3.A, U$4.1, U$4.2, U$9.1_+5V
- removed net N$3: U$5.3, U$6.+
- removed net N$5: C10.1, R27.2, U$7.2
- removed net N$6: C16.1, D3.1, R32.2, U$8.2
- removed net PENIRQ: R7.1, U$1.11
- removed net RD: X5.35
- removed net RST: R13.1, X5.9
- removed net VBAT: C12.1, C17.1, L2.1, R26.2, R28.2, R29.2, R30.2, S1.2
- new net +15V: C19.1, C20.1, D1.C, D4.C, R36.2
- new net BASE: R40.1, T1.1
- new net COLLECTOR: D5.K, T1.3
- new net DISPLAY_RESET: R13.1, X2.33, X5.9
- new net EMITTER: T1.2
- new net FB: C20.2, R36.1, R37.2, U$2.2
- new net IN_1: C21.2, U$3.1
- new net IR_RX: X2.36, X3.1
- new net IR_TX: R40.2, X2.38
- new net LX: D1.A, L1.2, U$2.5
- new net N$16: C21.1, D4.A, R38.2
- new net N$30: D5.A, R39.1
- new net N$35: LED4.C, R41.2
- new net N$36: LED5.C, R42.2
- new net OUT1_IN2: U$10.1, U$3.3
- new net OUT2: C23.2, U$10.3
- new net RANDOM: C23.1, X2.32
- new net STEPUP_ENABLE: U$2.1, X2.31
- new net VBAT+: U$4.+, U$5.3
- new net X1_RTC: Q3.1, U$5.1
- new net X2_RTC: Q3.4, U$5.2
- net +3V3: now also C14.1, C2.1, C3.1, C7.1, IC1.2, JMP1.1, R13.2, R14.2, R15.2, R2.2, R39.2, R6.2, U$6.1, X5.2, X5.3, X5.35, X5.4, X5.5, X5.6, X5.7, X5.8; no longer C1.1, C11.1, C5.1, IC2.8, R1.2, R3.2, R4.2, R5.2, U$5.8, U$7.3, X2.1, X2.17
- net +5V: now also C22.2, C6.1, C8.1, C9.1, L1.1, SJ2.2, U$10.4, U$2.3, U$3.4, U$9.1_+5V, X5.43; no longer D3.3, Q1.1
- net CE0: now also X5.38
- net D/C: now also JMP1.2
- net GND: now also C19.2, C22.1, C6.2, JMP1.3, R37.1, R38.1, R41.1, R42.1, U$10.2, U$2.4, U$3.2, U$4.GND, U$6.13, U$6.14, U$6.16, U$6.6, X3.2; no longer C10.2, C11.2, C15.2, C16.2, C17.2, D2.A, Q2.3, R10.1, R2.2, R31.1, R33.1, R7.2, SJ1.1, U$1.6, U$1.7, U$1.8, U$4.5, U$6.GND, U$7.1, U$7.4, U$7.6, U$7.EXP, U$8.4, U$8.9, U$8.GND, U$9.4_ID, U$9.GND3, U$9.GND4, X1.2, X5.6, X5.7, X5.8
- net GPIO19: now also LED4.A
- net GPIO26: now also LED5.A
- net INT: now also U$6.10; no longer U$7.5
- net MISO: no longer R35.1, U$1.12
- net MOSI: no longer R12.1, U$1.14
- net N$12: now also Q1.2; no longer Q2.2
- net N$20: now also Q1.1; no longer Q2.1
- net N$4: now also SJ2.1, X3.3; no longer R26.1, U$8.5
- net SCK: no longer U$1.16
- net SCL_3V3: now also R6.1, U$6.12; no longer U$7.7
- net SDA_3V3: now also R2.1, U$6.11; no longer U$7.8
- net TOUCH_X+: now also U$6.2; no longer U$1.2
- net TOUCH_X-: now also U$6.4; no longer U$1.4
- net TOUCH_Y+: now also U$6.3; no longer U$1.3
- net TOUCH_Y-: now also U$6.5; no longer U$1.5
- net VCC: now also C1.1, C5.1, IC2.8, R1.2, R3.2, R4.2, R5.2, U$5.8, X2.1, X2.17; no longer C14.1, C2.1, C3.1, C7.1, IC1.2, R12.2, R13.2, R14.2, R15.2, R34.2, R35.2, R6.2, U$1.1, U$1.10, U$1.9, X5.2, X5.3, X5.4, X5.5
Routing:
- net N$21: track 122.3 -> 0.00 mm, vias 1 -> 0
- net BAT+: track 100.7 -> 0.00 mm, vias 3 -> 0
- net N$3: track 83.8 -> 0.00 mm
- net ENABLE_STEPUP: track 81.2 -> 0.00 mm, vias 4 -> 0
- net RANDOM: track 0.00 -> 76.4 mm
- net IR_RX: track 0.00 -> 75.5 mm, vias 0 -> 1
- net STEPUP_ENABLE: track 0.00 -> 75.2 mm
- net +5V: track 102.1 -> 168.9 mm, vias 2 -> 0
- net +3V3: track 56.5 -> 119.5 mm
- net DISPLAY_RESET: track 0.00 -> 62.7 mm
- net IR_TX: track 0.00 -> 62.0 mm, vias 0 -> 1
- net GPIO19: track 0.00 -> 60.6 mm
- net GPIO26: track 0.00 -> 59.7 mm
- net N$28: track 52.8 -> 0.00 mm
- net VBAT: track 24.2 -> 0.00 mm
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Other:
- board size 85 x 86 mm -> 64.5 x 56 mm
- board text added: "20.5,0"
- board text added: "CrackberryPi v1.0.1"
- board text removed: "Connector"
- board text removed: "HDMI"
