File: Eagle/CrackberryPi.sch (EAGLE design)
At the start: 23 parts, among them IC1 X1205IS8, IC2 24C02CSM, J1 22-27-2031-03, Q1 MC-406, X1 1503_07, X2 057-040-1

Commit message: scherm en touchscreen bestanden en info
Parts:
- removed SJ1, SJ2: (no value), jumper:SJ
- added C6, C7: (no value), rcl:C-EUC0603
- added R7: 10k, rcl:R-EU_R0603
- added TP1_WP, TP2_WP: TPSTP15R, testpad:TPSTP15R
- added U$3: ADS7843, ads7843:ADS7843
- added WP_GND: (no value), jumper:SJ
- added X3: FH28-50S-0.5SH(51), con-hirose:FH28-50S-0.5SH(51)
Connections:
- removed net N$12: R6.2, SJ2.1
- new net INTERRUPT: R7.1, U$3.PENIRQ
- new net TOUCH_X+: U$3.X+
- new net TOUCH_X-: U$3.X-
- new net TOUCH_Y+: U$3.Y+
- new net TOUCH_Y-: U$3.Y-
- net +3V3: now also C6.1, C7.1, R6.2, R7.2, U$3.VCC, U$3.VREF; no longer SJ2.2
- net GND: now also C6.2, C7.2, TP1_WP.PP, U$3.GND, WP_GND.1; no longer SJ1.1
- net N$11: now also TP2_WP.PP, WP_GND.2; no longer SJ1.2
Other:
- note added: "FFC connector"
- note added: "HAT EEPROM"
- note added: "TOUCH"
- note removed: "HAT"
- moved on the sheet: C5, IC2, R4, R5, R6

Commit message: screen info
Parts:
- added C8, C9: (no value), rcl:C-EUC0603
- added LED1, LED2, LED3: (no value), eagle-ltspice:LED_ESML0603
- added Q2: FDN360P, transistor-power:FDN360P
- added R10: 1k, rcl:R-EU_R0603
- added R11, R8, R9: 470, rcl:R-EU_R0603
- added R12: THERMISTOR-5, varistor:THERMISTOR-5
- added R13, R14, R15, R16, R17, R24: 10k, rcl:R-EU_R0603
- added R18, R19, R20, R21, R22, R23: 147, rcl:R-EU_R0603
- added R25: 45k, rcl:R-EU_R0603
- added SV1: (no value), con-amp-mt:S02P
- added U$4: MCP73833, mcp73833:MCP73833
- added X4: MINI-USB-32005-301, con-cypressindustries:MINI-USB-32005-301
Connections:
- new net DE: R17.2
- new net H_SYNC: R15.1
- new net LEDK1: R18.2
- new net LEDK2: R19.2
- new net LEDK3: R20.2
- new net LEDK4: R21.2
- new net LEDK5: R22.2
- new net LEDK6: R23.2
- new net LED_ON: R24.2, R25.2
- new net N$12: Q2.S, R18.1, R19.1, R20.1, R21.1, R22.1, R23.1
- new net N$13: R8.2, U$4.STAT1
- new net N$14: LED1.C, R8.1
- new net N$15: R9.2, U$4.STAT2
- new net N$16: R11.2, U$4.PG
- new net N$17: LED3.C, R11.1
- new net N$18: LED2.C, R9.1
- new net N$19: R10.2, U$4.PROG
- new net N$20: Q2.G, R24.1
- new net N$21: R12.1, U$4.THERM
- new net N$22: C8.1, SV1-2.S, U$4.VBAT
- new net P_CLK: R16.2
- new net RST: R13.1
- new net V+: LED1.A, LED2.A, LED3.A, U$4.VDD, X4.1
- new net V_SYNC: R14.1
- net +3V3: now also R13.2, R14.2, R15.2, X3-2.1, X3-3.1, X3-4.1, X3-5.1
- net +5V: now also C9.1
- net GND: now also C8.2, C9.2, Q2.D, R10.1, R12.2, R16.1, R17.1, R25.1, SV1-1.S, U$4.VSS, X3-1.1, X3-14.1, X3-15.1, X3-16.1, X3-17.1, X3-18.1, X3-19.1, X3-20.1, X3-21.1, X3-22.1, X3-23.1, X3-24.1, X3-25.1, X3-26.1, X3-27.1, X3-28.1, X3-29.1, X3-30.1, X3-31.1, X3-32.1, X3-6.1, X3-7.1, X3-8.1, X4.5
Other:
- note added: "Li-ion charger"
- note added: "MCP73833/4"

Commit message: part selection
Parts:
- removed G1: CR2430H, battery:CR2430H
- removed IC1: X1205IS8, xicor:X1205IS8
- removed J1: 22-27-2031-03, con-molex:22-27-2031-03
- removed Q1: MC-406, crystal:MC-406
- removed TP1_WP, TP2_WP: TPSTP15R, testpad:TPSTP15R
- removed X1: 1503_07, con-lumberg:1503_07
- added Q3: (no value), crystal:CRYSTALMM20SS
- added R26: PC16SV, piher:PC16SV
- added U$5: MCP7940N, MCP7940N:MCP7940N
- added U$6: CR2032, cr2032:CR2032
- added WP_GND1: (no value), jumper:SJ
Connections:
- net GPIO10 renamed MOSI
- net GPIO14 renamed UART_TX
- net GPIO15 renamed UART_RX
- net GPIO9 renamed MISO
- removed net GPIO17: X2-11.S
- removed net GPIO4: X2-7.S
- removed net LED_ON: R24.2, R25.2
- removed net N$4: J1-1.S, X1.2
- removed net N$5: J1-2.S, X1.3
- removed net N$6: J1-3.S, X1.1
- new net ADDITIONAL_1: U$3.IN3
- new net ADDITIONAL_2: U$3.IN4
- new net N$23: R26.1A, R26.S2
- new net N$25: R26.1S
- new net PWM: R24.2, R25.2, X2-11.S
- net +3V3: now also U$5.VCC; no longer IC1.VCC
- net +5V: now also R26.S1
- net GND: now also R26.1E, U$5.VSS, U$6.-, WP_GND1.1; no longer G1.-, IC1.VSS, TP1_WP.PP
- net INT: now also U$5.INT, X2-7.S; no longer IC1.!IRQ
- net N$1: now also Q3.1, U$5.X2; no longer IC1.X1, Q1.2
- net N$11: no longer TP2_WP.PP
- net N$12: now also WP_GND1.2
- net N$2: now also Q3.2, U$5.X1; no longer IC1.X2, Q1.1
- net N$3: now also U$5.VBAT, U$6.+; no longer G1.+, IC1.VBACK
- net SCL_3V3: now also U$5.SCL; no longer IC1.SDL
- net SDA_3V3: now also U$5.SDA; no longer IC1.SDA
Other:
- note added: "BACKLIGHT"
- note added: "MCP7940N"
- note removed: "AUDIO"
- moved on the sheet: C1, C5, C6, C7, IC2, Q2, R1, R13, R14, R15, R16, R17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

Commit message: pcb development
Parts:
- removed C6: (no value), rcl:C-EUC0603
- removed D1: (no value), diode:ZENER-DIODESOD80C
- removed SV1: (no value), con-amp-mt:S02P
- removed U$2: MAX2650, MAX2650:MAX2650
- removed U$3: ADS7843, ads7843:ADS7843
- removed WP_GND, WP_GND1: (no value), jumper:SJ
- removed X3: FH28-50S-0.5SH(51), con-hirose:FH28-50S-0.5SH(51)
- removed X4: MINI-USB-32005-301, con-cypressindustries:MINI-USB-32005-301
- added C10: 1mf, rcl:C-EUC0603
- added C11: 10nf, rcl:C-EUC0603
- added C12, C13, C14, C15: 0.1mf, rcl:C-EUC0603
- added C16: 22mf, rcl:C-EUC0805
- added C17: 10mf, rcl:C-EUC0805
- added C18: (no value), rcl:C-EUC0603
- added D2: (no value), diode:ZENER-DIODESOD80C
- added D3: BAS40-05, diode:BAS40-05
- added IC1: REG1117, burr-brown:REG1117
- added L2: (no value), rcl:L-EUL4532P
- added Q1: (no value), semicon-smd-ipc:PNP-TRANSISTOR_SOT23
- added R27: 1k, rcl:R-EU_R0603
- added R28, R29, R34, R35: 10k, rcl:R-EU_R0603
- added R30, R32: 2m, rcl:R-EU_R0603
- added R31, R33: 220k, rcl:R-EU_R0603
- added S1: (no value), switch:255SB
- added SJ1: (no value), jumper:SJ
- added U$7: MAX17043, MAX17043:MAX17043
- added U$8: TPS61200, TPS61200:TPS61200
- added U$9: MICRO_USB, MICRO_USB:MICRO_USB
- added X1: 53261-02, con-molex:53261-02
- added X5: FH12-50S-0.5SH, FCI_62684:FH12-50S-0.5SH
- R12: value THERMISTOR-5 -> 10k; device varistor:THERMISTOR-5 -> rcl:R-EU_R0603
- R2: value (none) -> THERMISTOR-2,5; device rcl:R-EU_R0603 -> varistor:THERMISTOR-2,5
- R26: value PC16SV -> 10k; device piher:PC16SV -> rcl:R-EU_R0603
- R6: value 1k -> 10k
- U$1: value MAX2650 -> TSC2046; device MAX2650:MAX2650 -> tsc2046:TSC2046
Connections:
- net GPIO7 renamed CE1
- net GPIO8 renamed CE0
- removed net +15V: D1.C
- removed net ADDITIONAL_1: U$3.IN3
- removed net ADDITIONAL_2: U$3.IN4
- removed net GPIO11: X2-23.S
- removed net INTERRUPT: R7.1, U$3.PENIRQ
- removed net N$10: C3.1, D1.A, R2.2
- removed net N$11: IC2.WP, R6.1, WP_GND.2
- removed net N$16: R11.2, U$4.PG
- removed net N$25: R26.1S
- removed net N$7: U$1.OUT, U$2.IN
- removed net N$8: C3.2, U$1.IN
- removed net N$9: C2.1, U$2.OUT
- removed net RANDOM_OUTPUT: C2.2
- removed net V+: LED1.A, LED2.A, LED3.A, U$4.VDD, X4.1
- new net +5V/4: C9.1, X5-43.1
- new net 2046_BUSY: R34.1, U$1.BUSY
- new net 2046_CS: R6.1, U$1.CS
- new net BAT+: C8.1, R27.1, S1.S, U$4.VBAT, X1-1.S
- new net CS: X5-38.1
- new net D/C: X5-37.1
- new net ENABLE_STEPUP: Q1.E, R11.2, R28.1, U$4.PG, U$8.EN
- new net N$24: L2.2, U$8.L
- new net N$26: C15.1, U$8.VAUX
- new net N$27: R32.1, R33.2, U$8.FB
- new net N$28: D2.C, D3.A2, LED1.A, LED2.A, LED3.A, U$4.VDD, U$9.1_+5V
- new net N$4: R26.1, U$8.VIN
- new net N$5: C10.1, R27.2, U$7.CELL
- new net N$6: C16.1, D3.A1, R32.2, U$8.VOUT
- new net PENIRQ: R7.1, U$1.PENIRQ
- new net RD: X5-35.1
- new net SCK: U$1.DCLK, X2-23.S, X5-36.1
- new net VBAT: C12.1, C17.1, L2.1, R26.2, R28.2, R29.2, R30.2, S1.P
- new net VCC: C14.1, C2.1, C3.1, C7.1, IC1.VOUT, R12.2, R13.2, R14.2, R15.2, R34.2, R35.2, R6.2, U$1.IOVDD, U$1.VCC, U$1.VREF, X5-2.1, X5-3.1, X5-4.1, X5-5.1
- net +3V3: now also C11.1, U$7.VDD; no longer C6.1, C7.1, R13.2, R14.2, R15.2, R6.2, R7.2, U$3.VCC, U$3.VREF, X3-2.1, X3-3.1, X3-4.1, X3-5.1
- net +5V: now also C13.1, D3.C, IC1.VIN, Q1.B; no longer C4.1, C9.1, R26.S1, U$1.VCC, U$2.VCC
- net DE: now also X5-13.1
- net GND: now also C10.2, C11.2, C13.2, C14.2, C15.2, C16.2, C17.2, C18.1, C4.1, D2.A, IC1.GND, IC2.WP, Q1.C, R2.2, R31.1, R33.1, R7.2, SJ1.1, U$1.AUX, U$1.VBAT, U$7.CTG, U$7.EP, U$7.GND, U$7.QST_6, U$8.GND, U$9.4_ID, U$9.5_0V, U$9.GND, X1-2.S, X5-1.1, X5-14.1, X5-15.1, X5-16.1, X5-17.1, X5-18.1, X5-19.1, X5-20.1, X5-21.1, X5-22.1, X5-23.1, X5-24.1, X5-25.1, X5-26.1, X5-27.1, X5-28.1, X5-29.1, X5-30.1, X5-31.1, X5-32.1, X5-50.1, X5-6.1, X5-7.1, X5-8.1; no longer C4.2, C6.2, R12.2, R2.1, R26.1E, SV1-1.S, U$2.GND, U$3.GND, WP_GND.1, WP_GND1.1, X3-1.1, X3-14.1, X3-15.1, X3-16.1, X3-17.1, X3-18.1, X3-19.1, X3-20.1, X3-21.1, X3-22.1, X3-23.1, X3-24.1, X3-25.1, X3-26.1, X3-27.1, X3-28.1, X3-29.1, X3-30.1, X3-31.1, X3-32.1, X3-6.1, X3-7.1, X3-8.1, X4.5
- net H_SYNC: now also X5-11.1
- net INT: now also U$7.ALT_5
- net LEDK1: now also X5-44.1
- net LEDK2: now also X5-45.1
- net LEDK3: now also X5-46.1
- net LEDK4: now also X5-47.1
- net LEDK5: now also X5-48.1
- net LEDK6: now also X5-49.1
- net MISO: now also R35.1, U$1.DOUT, X5-33.1
- net MOSI: now also R12.1, U$1.DIN, X5-34.1
- net N$12: no longer WP_GND1.2
- net N$21: now also R2.1; no longer R12.1
- net N$22: now also R29.1, SJ1.2, U$8.PS; no longer C8.1, SV1-2.S, U$4.VBAT
- net N$23: now also C12.2, R30.1, R31.2, U$8.UVLD; no longer R26.1A, R26.S2
- net P_CLK: now also X5-12.1
- net RST: now also X5-9.1
- net SCL_3V3: now also U$7.SCL
- net SDA_3V3: now also U$7.SDA
- net TOUCH_X+: now also C2.2, U$1.X+, X5-39.1; no longer U$3.X+
- net TOUCH_X-: now also C18.2, U$1.X-, X5-41.1; no longer U$3.X-
- net TOUCH_Y+: now also C3.2, U$1.Y+, X5-42.1; no longer U$3.Y+
- net TOUCH_Y-: now also C4.2, U$1.Y-, X5-40.1; no longer U$3.Y-
- net V_SYNC: now also X5-10.1
Other:
- note added: "Fuel Gauge"
- note added: "LDO"
- note added: "Li+ charger"
- note added: "USB"
- note added: "battery"
- note added: "step_up"
- note removed: "Li-ion charger"
- note removed: "MCP73833/4"
- note removed: "RANDOM"
- moved on the sheet: C2, C3, C4, C7, C8, LED1, LED2, LED3, R10, R11, R6, R7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

Commit message: finalizing pcb first proto
schematics, library parts and gerber rar
Parts:
- removed C10: 1mf, rcl:C-EUC0603
- removed C11: 10nf, rcl:C-EUC0603
- removed C12, C15: 0.1mf, rcl:C-EUC0603
- removed C16: 22mf, rcl:C-EUC0805
- removed C17: 10mf, rcl:C-EUC0805
- removed D2: (no value), diode:ZENER-DIODESOD80C
- removed D3: BAS40-05, diode:BAS40-05
- removed L2: (no value), rcl:L-EUL4532P
- removed LED1, LED2, LED3: (no value), eagle-ltspice:LED_ESML0603
- removed Q2: FDN360P, transistor-power:FDN360P
- removed R10, R27: 1k, rcl:R-EU_R0603
- removed R11, R8, R9: 470, rcl:R-EU_R0603
- removed R12, R26, R28, R29, R34, R35, R7: 10k, rcl:R-EU_R0603
- removed R30, R32: 2m, rcl:R-EU_R0603
- removed R31, R33: 220k, rcl:R-EU_R0603
- removed S1: (no value), switch:255SB
- removed SJ1: (no value), jumper:SJ
- removed U$1: TSC2046, tsc2046:TSC2046
- removed U$7: MAX17043, MAX17043:MAX17043
- removed U$8: TPS61200, TPS61200:TPS61200
- removed X1: 53261-02, con-molex:53261-02
- added C19: 4.7mf, rcl:C-EUC0603
- added C20: 68pf, rcl:C-EUC0603
- added C21, C23: 470pf, rcl:C-EUC0603
- added C22: 0.1mf, rcl:C-EUC0603
- added C6: 10mf, rcl:C-EUC0603
- added D1: (no value), diode:DIODE-SOD123
- added D4: 1N759, diode:ZENER-DIODESOD80C
- added D5: SFH482, led:SFH482
- added JMP1: 0R-JUMPC, jump-0r-smd:0R-JUMPC
- added L1: 8.2mH, rcl:R-EU_R1210
- added LED4, LED5: (no value), eagle-ltspice:LED_ESML0603
- added R36: 1.3m, rcl:R-EU_R0603
- added R37: 110k, rcl:R-EU_R0603
- added R38, R39: 30, rcl:R-EU_R0603
- added R40: 1k, rcl:R-EU_R0603
- added R41, R42: 10k, rcl:R-EU_R0603
- added SJ2: (no value), jumper:SJ
- added T1: BC847, transistor:BC847
- added U$10, U$3: MAX2650, max2650:MAX2650
- added U$2: NCP1406, ncp1406:NCP1406
- added X3: C-GRID-03-70543, con-molex:C-GRID-03-70543
- C13, C14: value 0.1mf -> 4.7mF
- C8: value (none) -> 0.1mf
- C9: value (none) -> 1mf
- Q1: value (none) -> IRLML5203; device semicon-smd-ipc:PNP-TRANSISTOR_SOT23 -> transistor-power:IRLML5203
- R2: value THERMISTOR-2,5 -> 10k; device varistor:THERMISTOR-2,5 -> rcl:R-EU_R0603
- U$4: value MCP73833 -> CR1216; device mcp73833:MCP73833 -> cr1216:CR1216
- U$6: value CR2032 -> TSC2007; device cr2032:CR2032 -> tsc2046:TSC2007
Connections:
- net GPIO21 renamed AVALANCHE_ENABLE
- removed net +5V/4: C9.1, X5-43.1
- removed net 2046_BUSY: R34.1, U$1.BUSY
- removed net 2046_CS: R6.1, U$1.CS
- removed net BAT+: C8.1, R27.1, S1.S, U$4.VBAT, X1-1.S
- removed net CS: X5-38.1
- removed net ENABLE_STEPUP: Q1.E, R11.2, R28.1, U$4.PG, U$8.EN
- removed net GPIO12: X2-32.S
- removed net GPIO13: X2-33.S
- removed net GPIO16: X2-36.S
- removed net GPIO20: X2-38.S
- removed net GPIO6: X2-31.S
- removed net N$1: Q3.1, U$5.X2
- removed net N$13: R8.2, U$4.STAT1
- removed net N$14: LED1.C, R8.1
- removed net N$15: R9.2, U$4.STAT2
- removed net N$17: LED3.C, R11.1
- removed net N$18: LED2.C, R9.1
- removed net N$19: R10.2, U$4.PROG
- removed net N$2: Q3.2, U$5.X1
- removed net N$21: R2.1, U$4.THERM
- removed net N$22: R29.1, SJ1.2, U$8.PS
- removed net N$23: C12.2, R30.1, R31.2, U$8.UVLD
- removed net N$24: L2.2, U$8.L
- removed net N$26: C15.1, U$8.VAUX
- removed net N$27: R32.1, R33.2, U$8.FB
- removed net N$28: D2.C, D3.A2, LED1.A, LED2.A, LED3.A, U$4.VDD, U$9.1_+5V
- removed net N$3: U$5.VBAT, U$6.+
- removed net N$5: C10.1, R27.2, U$7.CELL
- removed net N$6: C16.1, D3.A1, R32.2, U$8.VOUT
- removed net PENIRQ: R7.1, U$1.PENIRQ
- removed net RD: X5-35.1
- removed net RST: R13.1, X5-9.1
- removed net VBAT: C12.1, C17.1, L2.1, R26.2, R28.2, R29.2, R30.2, S1.P
- new net +15V: C19.1, C20.1, D1.C, D4.C, R36.2
- new net BASE: R40.1, T1.B
- new net COLLECTOR: D5.C, T1.C
- new net DISPLAY_RESET: R13.1, X2-33.S, X5-9.1
- new net EMITTER: T1.E
- new net FB: C20.2, R36.1, R37.2, U$2.FB
- new net IN_1: C21.2, U$3.IN
- new net IR_RX: X2-36.S, X3-1.S
- new net IR_TX: R40.2, X2-38.S
- new net LX: D1.A, L1.2, U$2.LX
- new net N$16: C21.1, D4.A, R38.2
- new net N$30: D5.A, R39.1
- new net N$35: LED4.C, R41.2
- new net N$36: LED5.C, R42.2
- new net OUT1_IN2: U$10.IN, U$3.OUT
- new net OUT2: C23.2, U$10.OUT
- new net RANDOM: C23.1, X2-32.S
- new net STEPUP_ENABLE: U$2.CE, X2-31.S
- new net VBAT+: U$4.+, U$5.VBAT
- new net X1_RTC: Q3.1, U$5.X1
- new net X2_RTC: Q3.2, U$5.X2
- net +3V3: now also C14.1, C2.1, C3.1, C7.1, IC1.VOUT, JMP1-0R.1, R13.2, R14.2, R15.2, R2.2, R39.2, R6.2, U$6.VDD, X5-2.1, X5-3.1, X5-35.1, X5-4.1, X5-5.1, X5-6.1, X5-7.1, X5-8.1; no longer C1.1, C11.1, C5.1, IC2.VCC, R1.2, R3.2, R4.2, R5.2, U$5.VCC, U$7.VDD, X2-1.S, X2-17.S
- net +5V: now also C22.2, C6.1, C8.1, C9.1, L1.1, SJ2.2, U$10.VCC, U$2.VDD, U$3.VCC, U$9.1_+5V, X5-43.1; no longer D3.C, Q1.B
- net CE0: now also X5-38.1
- net D/C: now also JMP1-0R.2
- net GND: now also C19.2, C22.1, C6.2, JMP1-0R.3, Q1.D, R37.1, R38.1, R41.1, R42.1, U$10.GND, U$2.GND, U$3.GND, U$4.-, U$6.A0, U$6.A1, U$6.AUX, U$6.GND, X3-2.S; no longer C10.2, C11.2, C15.2, C16.2, C17.2, D2.A, Q1.C, Q2.D, R10.1, R2.2, R31.1, R33.1, R7.2, SJ1.1, U$1.AUX, U$1.GND, U$1.VBAT, U$4.VSS, U$6.-, U$7.CTG, U$7.EP, U$7.GND, U$7.QST_6, U$8.GND, U$9.4_ID, X1-2.S, X5-6.1, X5-7.1, X5-8.1
- net GPIO19: now also LED4.A
- net GPIO26: now also LED5.A
- net INT: now also U$6.INT; no longer U$7.ALT_5
- net MISO: no longer R35.1, U$1.DOUT
- net MOSI: no longer R12.1, U$1.DIN
- net N$12: now also Q1.S; no longer Q2.S
- net N$20: now also Q1.G; no longer Q2.G
- net N$4: now also SJ2.1, X3-3.S; no longer R26.1, U$8.VIN
- net SCK: no longer U$1.DCLK
- net SCL_3V3: now also R6.1, U$6.SCL; no longer U$7.SCL
- net SDA_3V3: now also R2.1, U$6.SDA; no longer U$7.SDA
- net TOUCH_X+: now also U$6.X+; no longer U$1.X+
- net TOUCH_X-: now also U$6.X-; no longer U$1.X-
- net TOUCH_Y+: now also U$6.Y+; no longer U$1.Y+
- net TOUCH_Y-: now also U$6.Y-; no longer U$1.Y-
- net VCC: now also C1.1, C5.1, IC2.VCC, R1.2, R3.2, R4.2, R5.2, U$5.VCC, X2-1.S, X2-17.S; no longer C14.1, C2.1, C3.1, C7.1, IC1.VOUT, R12.2, R13.2, R14.2, R15.2, R34.2, R35.2, R6.2, U$1.IOVDD, U$1.VCC, U$1.VREF, X5-2.1, X5-3.1, X5-4.1, X5-5.1
Other:
- note added: "Vout=1.19(R1/R2+1)"
- note removed: "Fuel Gauge"
- note removed: "Li+ charger"
- note removed: "battery"
- note removed: "step_up"
- moved on the sheet: C13, C14, C18, C2, C3, C4, C7, C8, C9, IC1, Q3, R13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
