File: Eagle/CrackberryPi_1.0.2.brd (EAGLE design)
At the start: 85 x 96 mm, 131 parts, among them IC1 REG1117, IC2 24C02CSM, Q1 IRLML5203, T1 BC847, X1 53261-02, X3 C-GRID-03-70543, X5 FH12-50S-0.5SH

Commit message: documentatie pcb
Parts:
- moved R3 0.95 mm to (72.1, 49.6)
- moved R1 0.65 mm to (69.0, 51.2)
- moved R39 0.60 mm to (60.1, 92.6)
- moved R12 0.41 mm to (68.2, 92.2)
- moved LED1 0.40 mm to (67.4, 94.7)
Routing:
- net COL1: track 104.7 -> 115.6 mm
- net N$30: track 7.40 -> 6.80 mm
- net +3V3: track 186.2 -> 186.8 mm
Other:
- board text added: "10uF"
- board text added: "1K"
- board text added: "1uF"
- board text added: "2x 3.9K"
- board text added: "317R"
- board text added: "3x 10K"
- board text added: "3x 4.7uF"
- board text added: "45K"
- board text added: "47pF"
- board text added: "609-1202-1-ND ZIF-50"
- board text added: "6x 147R"
- board text added: "BAT-HLD-012 CR1216"
- board text added: "BC847"
- board text added: "BQ24297"
- board text added: "CAT24C32"
- board text added: "CM200C 32.768kHz"
- board text added: "IRLML5203 MOSFET"
- board text added: "LED"
- board text added: "MCP7940"
- board text added: "SFH482"
- board text added: "TCA8424"
- board text added: "TSOP38238"
- board text added: "uUSB-B"

Commit message: pictures, pcb advancements
Parts:
- added TP1, TP2: TPTP20SQ, testpad:TP20SQ
- moved C7 1.37 mm to (27.1, 63.0), turned to 0 degrees
- moved C23 1.03 mm to (23.5, 66.1)
- moved R7 0.64 mm to (82.0, 39.1)
- moved SJ2 0.45 mm to (78.7, 47.0)
- moved X3 0.40 mm to (82.7, 50.5)
Connections:
- net GND: now also TP2.TP
- net N$3: now also TP1.TP
Routing:
- net SCL_3V3: track 189.3 -> 166.4 mm
- net SDA_3V3: track 183.6 -> 163.1 mm
- net N$3: track 8.80 -> 27.8 mm
- net INT: track 178.6 -> 171.1 mm
- net COL1: track 115.6 -> 122.3 mm
- net IR_RX: track 60.7 -> 63.2 mm
- net VCC: track 74.9 -> 76.9 mm
- net STEPUP_ENABLE: track 75.9 -> 77.7 mm
- net ID_SD: track 28.7 -> 30.2 mm
- net +3V3: track 186.8 -> 187.9 mm
- net ID_SC: track 29.8 -> 30.9 mm
- net DISPLAY_RESET: track 79.6 -> 80.5 mm
- net +5V: track 210.5 -> 211.3 mm
- net GND: track 117.9 -> 117.2 mm, vias 11 -> 8
- net ROW9: track 42.1 -> 41.4 mm
- added copper zone on layer 1, net +5V
Other:
- board text added: "+"
