File: Eagle/CrackberryPi_1.0.2.sch (EAGLE design)
At the start: 131 parts, among them IC1 REG1117, IC2 24C02CSM, Q1 IRLML5203, T1 BC847, X1 53261-02, X3 C-GRID-03-70543, X5 FH12-50S-0.5SH

Commit message: pictures, pcb advancements
Parts:
- added TP1, TP2: TPTP20SQ, testpad:TPTP20SQ
Connections:
- net GND: now also TP2.TP
- net N$3: now also TP1.TP
Changed lines of the file:
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@@
 <part name="FN-RIGHT" library="DOME" deviceset="DOME" device=""/>
 <part name="P+5" library="supply1" deviceset="VCC" device=""/>
+<part name="TP1" library="testpad" deviceset="TP" device="TP20SQ"/>
+<part name="TP2" library="testpad" deviceset="TP" device="TP20SQ"/>
 </parts>
 <sheets>
@@
 <instance part="FN-RIGHT" gate="G$1" x="1513.84" y="114.3"/>
 <instance part="P+5" gate="VCC" x="695.96" y="320.04"/>
+<instance part="TP1" gate="G$1" x="-45.72" y="160.02"/>
+<instance part="TP2" gate="G$1" x="-43.18" y="152.4" rot="R180"/>
 </instances>
 <busses>
@@
 <wire x1="-58.42" y1="149.86" x2="-50.8" y2="149.86" width="0.1524" layer="91"/>
 <junction x="-58.42" y="149.86"/>
+<pinref part="TP2" gate="G$1" pin="TP"/>
+<junction x="-43.18" y="154.94"/>
 </segment>
 <segment>
@@
 <junction x="-58.42" y="157.48"/>
 <wire x1="-83.82" y1="157.48" x2="-58.42" y2="157.48" width="0.1524" layer="91"/>
-<wire x1="-43.18" y1="157.48" x2="-58.42" y2="157.48" width="0.1524" layer="91"/>
-</segment>
-</net>
+<wire x1="-43.18" y1="157.48" x2="-45.72" y2="157.48" width="0.1524" layer="91"/>
+<pinref part="TP1" gate="G$1" pin="TP"/>
+<wire x1="-45.72" y1="157.48" x2="-58.42" y2="157.48" width="0.1524" layer="91"/>
+<junction x="-45.72" y="157.48"/>
+</segment>
+</net>
