File: Eagle/CrackberryPi_1.0.4.brd (EAGLE design)
At the start: 85 x 96 mm, 149 parts, among them IC1 REG1117, IC2 24C02CSM, Q1 IRLML5203, Q2 32.768, T1 BC847, X1 53261-02, X3 C-GRID-03-70543, X5 FH12-50S-0.5SH

Commit message: BOM en IR
Parts:
- moved TP2 9.36 mm to (82.6, 13.2)
- moved SJ2 6.86 mm to (77.7, 39.4), turned to 180 degrees
- moved TP1 1.82 mm to (82.7, 10.2)
- moved C9 1.45 mm to (44.4, 50.4)
- moved Q3 0.20 mm to (76.7, 51.4)
Routing:
- net SDA_3V3: track 239.9 -> 245.6 mm, vias 7 -> 6
- net INT: track 171.4 -> 176.4 mm
- net SCK: track 76.1 -> 71.6 mm
- net GPIO27: track 32.4 -> 28.4 mm
- net N$6: track 52.3 -> 48.4 mm, vias 1 -> 0
- net GPIO23: track 40.7 -> 37.0 mm
- net SCL_3V3: track 221.7 -> 218.1 mm
- net +5V: track 208.4 -> 211.5 mm
- net N$3: track 104.3 -> 107.2 mm, vias 2 -> 3
- net GPIO22: track 35.6 -> 32.7 mm
- net GPIO24: track 44.1 -> 41.3 mm
- net PWM: track 38.3 -> 36.5 mm
- net GPIO25: track 45.9 -> 44.2 mm
- net MISO: track 79.2 -> 77.6 mm
- net IR_RX: track 63.1 -> 61.8 mm
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
Commit message: screen documentation
Parts:
- added GD, ID-SC, ID-SD, INT, SCL, SDA, V33, V5, VCC: TPB1,27, testpad:B1,27
- moved C15 6.15 mm to (73.0, 78.0), turned to 270 degrees
- moved ANTENNA 4.35 mm to (28.2, 93.5)
- moved L3 3.61 mm to (27.4, 89.2)
- moved U$4 2.27 mm to (67.5, 70.0)
- moved X5 1.00 mm to (48.0, 53.2)
- moved C5 0.99 mm to (53.7, 52.6), turned to 90 degrees
- moved C3 0.87 mm to (38.5, 56.2), turned to 90 degrees
- moved C18 0.20 mm to (38.8, 58.6)
Connections:
- new net V+: C5.1, IC2.8, R4.2, R5.2, SV1.17, VCC.TP
- net +3V3: now also V33.TP
- net +5V: now also V5.TP
- net GND: now also GD.TP
- net ID_SC: now also ID-SC.TP
- net ID_SD: now also ID-SD.TP
- net INT: now also INT.TP
- net SCL_3V3: now also SCL.TP
- net SDA_3V3: now also SDA.TP
- net VCC: no longer C5.1, IC2.8, R4.2, R5.2, SV1.17
Routing:
- net +5V: track 211.5 -> 239.5 mm
- net SDA_3V3: track 245.6 -> 218.1 mm, vias 6 -> 7
- net VCC: track 80.1 -> 55.9 mm
- net V+: track 0.00 -> 22.9 mm, vias 0 -> 1
- net INT: track 176.4 -> 165.9 mm, vias 5 -> 6
- net SCL_3V3: track 218.1 -> 208.5 mm, vias 9 -> 10
- net FM_RST: track 72.9 -> 63.8 mm
- net ID_SD: track 30.2 -> 36.2 mm
- net PWM: track 36.5 -> 42.4 mm, vias 1 -> 2
- net MISO: track 77.6 -> 83.4 mm
- net +3V3: track 226.5 -> 232.2 mm, vias 9 -> 10
- net N$3: track 107.2 -> 101.6 mm
- net GPIO22: track 32.7 -> 37.8 mm
- net N$25: track 17.6 -> 21.6 mm
- net ID_SC: track 30.9 -> 34.9 mm, vias 0 -> 1
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Other:
- outline, holes or cut-outs redrawn
