File: Eagle/CrackberryPi_1.0.4.sch (EAGLE design)
At the start: 149 parts, among them IC1 REG1117, IC2 24C02CSM, Q1 IRLML5203, Q2 32.768, T1 BC847, X1 53261-02, X3 C-GRID-03-70543, X5 FH12-50S-0.5SH

Commit message: BOM en IR
Other:
- moved on the sheet: C24, C25, C26, C8, Q2
Changed lines of the file:
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@@
 <instance part="AUDIO_R" gate="G$1" x="576.58" y="246.38"/>
 <instance part="GND1" gate="1" x="571.5" y="220.98"/>
-<instance part="Q2" gate="G$1" x="500.38" y="193.04"/>
+<instance part="Q2" gate="G$1" x="508" y="193.04"/>
 <instance part="U$8" gate="G$1" x="535.94" y="152.4"/>
-<instance part="C8" gate="G$1" x="492.76" y="182.88"/>
-<instance part="C24" gate="G$1" x="513.08" y="180.34" rot="R180"/>
-<instance part="GND43" gate="1" x="492.76" y="170.18"/>
-<instance part="GND44" gate="1" x="513.08" y="170.18"/>
+<instance part="C8" gate="G$1" x="500.38" y="182.88"/>
+<instance part="C24" gate="G$1" x="515.62" y="180.34" rot="R180"/>
+<instance part="GND43" gate="1" x="500.38" y="170.18"/>
+<instance part="GND44" gate="1" x="515.62" y="170.18"/>
 <instance part="GND45" gate="1" x="513.08" y="149.86" rot="R270"/>
-<instance part="C25" gate="G$1" x="563.88" y="187.96"/>
-<instance part="C26" gate="G$1" x="576.58" y="187.96"/>
+<instance part="C25" gate="G$1" x="556.26" y="182.88"/>
+<instance part="C26" gate="G$1" x="574.04" y="182.88"/>
 <instance part="GND46" gate="1" x="579.12" y="142.24"/>
 <instance part="C27" gate="G$1" x="591.82" y="137.16"/>
@@
 <pinref part="C8" gate="G$1" pin="2"/>
 <pinref part="GND43" gate="1" pin="GND"/>
-<wire x1="492.76" y1="177.8" x2="492.76" y2="172.72" width="0.1524" layer="91"/>
+<wire x1="500.38" y1="177.8" x2="500.38" y2="172.72" width="0.1524" layer="91"/>
 </segment>
 <segment>
 <pinref part="C24" gate="G$1" pin="1"/>
 <pinref part="GND44" gate="1" pin="GND"/>
-<wire x1="513.08" y1="177.8" x2="513.08" y2="172.72" width="0.1524" layer="91"/>
+<wire x1="515.62" y1="177.8" x2="515.62" y2="172.72" width="0.1524" layer="91"/>
 </segment>
 <segment>
@@
 <pinref part="SV3" gate="1" pin="2"/>
 <wire x1="485.14" y1="358.14" x2="495.3" y2="358.14" width="0.1524" layer="91"/>
-<label x="487.68" y="358.14" size="1.778" layer="95"/>
+<label x="492.76" y="358.14" size="1.778" layer="95"/>
 </segment>
 </net>
@@
 <segment>
 <pinref part="U$8" gate="G$1" pin="SCLK"/>
-<wire x1="541.02" y1="124.46" x2="541.02" y2="104.14" width="0.1524" layer="91"/>
-<label x="541.02" y="104.14" size="1.778" layer="95" rot="R90"/>
+<wire x1="541.02" y1="124.46" x2="541.02" y2="109.22" width="0.1524" layer="91"/>
+<wire x1="541.02" y1="109.22" x2="528.32" y2="109.22" width="0.1524" layer="91"/>
+<label x="528.32" y="109.22" size="1.778" layer="95"/>
 </segment>
 <segment>
 <pinref part="SV3" gate="1" pin="6"/>
 <wire x1="485.14" y1="363.22" x2="495.3" y2="363.22" width="0.1524" layer="91"/>
-<label x="487.68" y="363.22" size="1.778" layer="95"/>
+<label x="492.76" y="363.22" size="1.778" layer="95"/>
 </segment>
 </net>
@@
 <segment>
 <pinref part="U$8" gate="G$1" pin="SDIO"/>
-<wire x1="546.1" y1="124.46" x2="546.1" y2="104.14" width="0.1524" layer="91"/>
-<label x="546.1" y="104.14" size="1.778" layer="95" rot="R90"/>
+<wire x1="546.1" y1="124.46" x2="546.1" y2="106.68" width="0.1524" layer="91"/>
+<wire x1="546.1" y1="106.68" x2="528.32" y2="106.68" width="0.1524" layer="91"/>
+<label x="528.32" y="106.68" size="1.778" layer="95"/>
 </segment>
 <segment>
 <pinref part="SV3" gate="1" pin="4"/>
 <wire x1="485.14" y1="360.68" x2="495.3" y2="360.68" width="0.1524" layer="91"/>
-<label x="487.68" y="360.68" size="1.778" layer="95"/>
+<label x="492.76" y="360.68" size="1.778" layer="95"/>
 </segment>
 </net>
@@
 <wire x1="469.9" y1="370.84" x2="459.74" y2="370.84" width="0.1524" layer="91"/>
 <pinref part="SV3" gate="1" pin="11"/>
-<label x="459.74" y="370.84" size="1.778" layer="95"/>
+<label x="457.2" y="370.84" size="1.778" layer="95"/>
 </segment>
 </net>
@@
 <wire x1="469.9" y1="368.3" x2="459.74" y2="368.3" width="0.1524" layer="91"/>
 <pinref part="SV3" gate="1" pin="9"/>
-<label x="459.74" y="368.3" size="1.778" layer="95"/>
+<label x="457.2" y="368.3" size="1.778" layer="95"/>
 </segment>
 </net>
@@
 <pinref part="SV3" gate="1" pin="3"/>
 <wire x1="469.9" y1="360.68" x2="459.74" y2="360.68" width="0.1524" layer="91"/>
-<label x="459.74" y="360.68" size="1.778" layer="95"/>
+<label x="457.2" y="360.68" size="1.778" layer="95"/>
 </segment>
 </net>
@@
 <pinref part="SV3" gate="1" pin="1"/>
 <wire x1="469.9" y1="358.14" x2="459.74" y2="358.14" width="0.1524" layer="91"/>
-<label x="459.74" y="358.14" size="1.778" layer="95"/>
+<label x="457.2" y="358.14" size="1.778" layer="95"/>
 </segment>
 </net>
@@
 <segment>
 <wire x1="469.9" y1="373.38" x2="459.74" y2="373.38" width="0.1524" layer="91"/>
-<label x="459.74" y="373.38" size="1.778" layer="95"/>
+<label x="457.2" y="373.38" size="1.778" layer="95"/>
 <pinref part="SV3" gate="1" pin="13"/>
 </segment>
@@
 <pinref part="SV3" gate="1" pin="7"/>
 <wire x1="469.9" y1="365.76" x2="454.66" y2="365.76" width="0.1524" layer="91"/>
-<label x="459.74" y="365.76" size="1.778" layer="95"/>
 <pinref part="+3V24" gate="G$1" pin="+3V3"/>
 <wire x1="454.66" y1="368.3" x2="454.66" y2="365.76" width="0.1524" layer="91"/>
@@
 <segment>
 <pinref part="C25" gate="G$1" pin="1"/>
-<wire x1="563.88" y1="190.5" x2="563.88" y2="200.66" width="0.1524" layer="91"/>
-<label x="558.8" y="200.66" size="1.778" layer="95"/>
+<wire x1="556.26" y1="185.42" x2="556.26" y2="193.04" width="0.1524" layer="91"/>
+<label x="556.26" y="193.04" size="1.778" layer="95"/>
 </segment>
 </net>
@@
 <segment>
 <pinref part="C26" gate="G$1" pin="1"/>
-<wire x1="576.58" y1="190.5" x2="576.58" y2="200.66" width="0.1524" layer="91"/>
-<label x="571.5" y="200.66" size="1.778" layer="95"/>
+<wire x1="574.04" y1="185.42" x2="574.04" y2="193.04" width="0.1524" layer="91"/>
+<label x="574.04" y="193.04" size="1.778" layer="95"/>
 </segment>
 </net>
@@
 <pinref part="Q2" gate="G$1" pin="2"/>
 <wire x1="551.18" y1="175.26" x2="551.18" y2="193.04" width="0.1524" layer="91"/>
-<wire x1="551.18" y1="193.04" x2="513.08" y2="193.04" width="0.1524" layer="91"/>
+<wire x1="551.18" y1="193.04" x2="515.62" y2="193.04" width="0.1524" layer="91"/>
 <pinref part="C24" gate="G$1" pin="2"/>
-<wire x1="513.08" y1="193.04" x2="502.92" y2="193.04" width="0.1524" layer="91"/>
-<wire x1="513.08" y1="193.04" x2="513.08" y2="185.42" width="0.1524" layer="91"/>
-<junction x="513.08" y="193.04"/>
+<wire x1="515.62" y1="193.04" x2="510.54" y2="193.04" width="0.1524" layer="91"/>
+<wire x1="515.62" y1="193.04" x2="515.62" y2="185.42" width="0.1524" layer="91"/>
+<junction x="515.62" y="193.04"/>
 </segment>
 </net>
@@
 <pinref part="Q2" gate="G$1" pin="1"/>
 <pinref part="C8" gate="G$1" pin="1"/>
-<wire x1="497.84" y1="193.04" x2="492.76" y2="193.04" width="0.1524" layer="91"/>
-<wire x1="492.76" y1="193.04" x2="492.76" y2="185.42" width="0.1524" layer="91"/>
+<wire x1="505.46" y1="193.04" x2="500.38" y2="193.04" width="0.1524" layer="91"/>
+<wire x1="500.38" y1="193.04" x2="500.38" y2="185.42" width="0.1524" layer="91"/>
 <pinref part="U$8" gate="G$1" pin="RCLK"/>
-<wire x1="551.18" y1="124.46" x2="551.18" y2="93.98" width="0.1524" layer="91"/>
-<wire x1="551.18" y1="93.98" x2="487.68" y2="93.98" width="0.1524" layer="91"/>
-<wire x1="487.68" y1="93.98" x2="487.68" y2="193.04" width="0.1524" layer="91"/>
-<wire x1="487.68" y1="193.04" x2="492.76" y2="193.04" width="0.1524" layer="91"/>
-<junction x="492.76" y="193.04"/>
+<wire x1="551.18" y1="124.46" x2="551.18" y2="104.14" width="0.1524" layer="91"/>
+<wire x1="551.18" y1="104.14" x2="492.76" y2="104.14" width="0.1524" layer="91"/>
+<wire x1="492.76" y1="104.14" x2="492.76" y2="193.04" width="0.1524" layer="91"/>
+<wire x1="492.76" y1="193.04" x2="500.38" y2="193.04" width="0.1524" layer="91"/>
+<junction x="500.38" y="193.04"/>
 </segment>
 </net>
@@
 <pinref part="C25" gate="G$1" pin="2"/>
 <pinref part="U$8" gate="G$1" pin="LIN"/>
-<wire x1="563.88" y1="182.88" x2="556.26" y2="182.88" width="0.1524" layer="91"/>
-<wire x1="556.26" y1="182.88" x2="556.26" y2="175.26" width="0.1524" layer="91"/>
+<wire x1="556.26" y1="177.8" x2="556.26" y2="175.26" width="0.1524" layer="91"/>
 </segment>
 </net>
@@
 <pinref part="C26" gate="G$1" pin="2"/>
 <pinref part="U$8" gate="G$1" pin="RIN"/>
-<wire x1="576.58" y1="182.88" x2="576.58" y2="160.02" width="0.1524" layer="91"/>
-<wire x1="576.58" y1="160.02" x2="571.5" y2="160.02" width="0.1524" layer="91"/>
-</segment>
-</net>
+<wire x1="574.04" y1="177.8" x2="574.04" y2="160.02" width="0.1524" layer="91"/>
+<wire x1="574.04" y1="160.02" x2="571.5" y2="160.02" width="0.1524" layer="91"/>
+</segment>
+</net>

Commit message: screen documentation
Parts:
- added GD, ID-SC, ID-SD, INT, SCL, SDA, V33, V5, VCC: TPB1,27, testpad:TPB1,27
Connections:
- new net V+: C5.1, IC2.VCC, R4.2, R5.2, SV1.17, VCC.TP
- net +3V3: now also V33.TP
- net +5V: now also V5.TP
- net GND: now also GD.TP
- net ID_SC: now also ID-SC.TP
- net ID_SD: now also ID-SD.TP
- net INT: now also INT.TP
- net SCL_3V3: now also SCL.TP
- net SDA_3V3: now also SDA.TP
- net VCC: no longer C5.1, IC2.VCC, R4.2, R5.2, SV1.17
Changed lines of the file:
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@@
 <part name="P+21" library="supply1" deviceset="+5V" device=""/>
 <part name="P+23" library="supply1" deviceset="VCC" device=""/>
-<part name="P+24" library="supply1" deviceset="VCC" device=""/>
 <part name="P+25" library="supply1" deviceset="VCC" device=""/>
 <part name="P+26" library="supply1" deviceset="VCC" device=""/>
 <part name="P+27" library="supply1" deviceset="VCC" device=""/>
 <part name="P+28" library="supply1" deviceset="VCC" device=""/>
-<part name="P+30" library="supply1" deviceset="VCC" device=""/>
-<part name="P+31" library="supply1" deviceset="VCC" device=""/>
-<part name="P+32" library="supply1" deviceset="VCC" device=""/>
-<part name="P+33" library="supply1" deviceset="VCC" device=""/>
 <part name="+3V2" library="supply1" deviceset="+3V3" device=""/>
 <part name="+3V3" library="supply1" deviceset="+3V3" device=""/>
@@
 <part name="GND62" library="supply1" deviceset="GND" device=""/>
 <part name="P+9" library="supply1" deviceset="+5V" device=""/>
+<part name="SDA" library="testpad" deviceset="TP" device="B1,27"/>
+<part name="SCL" library="testpad" deviceset="TP" device="B1,27"/>
+<part name="INT" library="testpad" deviceset="TP" device="B1,27"/>
+<part name="ID-SC" library="testpad" deviceset="TP" device="B1,27"/>
+<part name="ID-SD" library="testpad" deviceset="TP" device="B1,27"/>
+<part name="GD" library="testpad" deviceset="TP" device="B1,27"/>
+<part name="VCC" library="testpad" deviceset="TP" device="B1,27"/>
+<part name="V5" library="testpad" deviceset="TP" device="B1,27"/>
+<part name="V33" library="testpad" deviceset="TP" device="B1,27"/>
+<part name="SUPPLY1" library="supply2" deviceset="V+" device=""/>
+<part name="SUPPLY2" library="supply2" deviceset="V+" device=""/>
+<part name="SUPPLY3" library="supply2" deviceset="V+" device=""/>
+<part name="SUPPLY4" library="supply2" deviceset="V+" device=""/>
+<part name="SUPPLY5" library="supply2" deviceset="V+" device=""/>
 </parts>
 <sheets>
@@
 <instance part="P+21" gate="1" x="149.86" y="304.8"/>
 <instance part="P+23" gate="VCC" x="-30.48" y="393.7"/>
-<instance part="P+24" gate="VCC" x="-20.32" y="373.38"/>
 <instance part="P+25" gate="VCC" x="-66.04" y="396.24"/>
 <instance part="P+26" gate="VCC" x="-73.66" y="396.24"/>
 <instance part="P+27" gate="VCC" x="-83.82" y="401.32"/>
 <instance part="P+28" gate="VCC" x="-149.86" y="396.24"/>
-<instance part="P+30" gate="VCC" x="-119.38" y="332.74"/>
-<instance part="P+31" gate="VCC" x="-96.52" y="332.74"/>
-<instance part="P+32" gate="VCC" x="-86.36" y="332.74"/>
-<instance part="P+33" gate="VCC" x="-66.04" y="304.8"/>
 <instance part="+3V2" gate="G$1" x="149.86" y="398.78"/>
 <instance part="+3V3" gate="G$1" x="160.02" y="398.78"/>
@@
 <instance part="GND62" gate="1" x="449.58" y="363.22" rot="R270"/>
 <instance part="P+9" gate="1" x="-50.8" y="193.04"/>
+<instance part="SDA" gate="G$1" x="0" y="388.62"/>
+<instance part="SCL" gate="G$1" x="0" y="386.08"/>
+<instance part="INT" gate="G$1" x="0" y="383.54"/>
+<instance part="ID-SC" gate="G$1" x="15.24" y="358.14"/>
+<instance part="ID-SD" gate="G$1" x="0" y="358.14"/>
+<instance part="GD" gate="G$1" x="0" y="381"/>
+<instance part="VCC" gate="G$1" x="-17.78" y="370.84"/>
+<instance part="V5" gate="G$1" x="-7.62" y="187.96"/>
+<instance part="V33" gate="G$1" x="17.78" y="187.96"/>
+<instance part="SUPPLY1" gate="1" x="-20.32" y="373.38"/>
+<instance part="SUPPLY2" gate="1" x="-119.38" y="332.74"/>
+<instance part="SUPPLY3" gate="1" x="-96.52" y="332.74"/>
+<instance part="SUPPLY4" gate="1" x="-86.36" y="332.74"/>
+<instance part="SUPPLY5" gate="1" x="-66.04" y="304.8"/>
 </instances>
 <busses>
@@
 <pinref part="SV1" gate="G$1" pin="9"/>
 <wire x1="-27.94" y1="378.46" x2="0" y2="378.46" width="0.1524" layer="91"/>
+<pinref part="GD" gate="G$1" pin="TP"/>
+<junction x="0" y="378.46"/>
 </segment>
 <segment>
@@
 <wire x1="-83.82" y1="381" x2="0" y2="381" width="0.1524" layer="91"/>
 <pinref part="SV1" gate="G$1" pin="7"/>
+<pinref part="INT" gate="G$1" pin="TP"/>
+<junction x="0" y="381"/>
 </segment>
 <segment>
@@
 <pinref part="SV1" gate="G$1" pin="5"/>
 <wire x1="-15.24" y1="383.54" x2="0" y2="383.54" width="0.1524" layer="91"/>
+<pinref part="SCL" gate="G$1" pin="TP"/>
+<junction x="0" y="383.54"/>
 </segment>
 <segment>
@@
 <pinref part="SV1" gate="G$1" pin="3"/>
 <wire x1="-15.24" y1="386.08" x2="0" y2="386.08" width="0.1524" layer="91"/>
+<pinref part="SDA" gate="G$1" pin="TP"/>
+<junction x="0" y="386.08"/>
 </segment>
 <segment>
@@
 <pinref part="P+9" gate="1" pin="+5V"/>
 <wire x1="-50.8" y1="190.5" x2="-50.8" y2="185.42" width="0.1524" layer="91"/>
+<pinref part="V5" gate="G$1" pin="TP"/>
+<junction x="-7.62" y="185.42"/>
 </segment>
 <segment>
@@
 <pinref part="SV1" gate="G$1" pin="27"/>
 <wire x1="0" y1="355.6" x2="-15.24" y2="355.6" width="0.1524" layer="91"/>
+<pinref part="ID-SD" gate="G$1" pin="TP"/>
+<junction x="0" y="355.6"/>
 </segment>
 <segment>
@@
 <pinref part="SV1" gate="G$1" pin="28"/>
 <wire x1="27.94" y1="355.6" x2="15.24" y2="355.6" width="0.1524" layer="91"/>
+<pinref part="ID-SC" gate="G$1" pin="TP"/>
+<junction x="15.24" y="355.6"/>
 </segment>
 <segment>
@@
 <net name="VCC" class="0">
 <segment>
-<pinref part="R4" gate="G$1" pin="2"/>
-<pinref part="P+30" gate="VCC" pin="VCC"/>
-<wire x1="-119.38" y1="330.2" x2="-119.38" y2="322.58" width="0.1524" layer="91"/>
-</segment>
-<segment>
-<pinref part="IC2" gate="G$1" pin="VCC"/>
-<wire x1="-96.52" y1="330.2" x2="-96.52" y2="314.96" width="0.1524" layer="91"/>
-<pinref part="P+31" gate="VCC" pin="VCC"/>
-</segment>
-<segment>
-<pinref part="R5" gate="G$1" pin="2"/>
-<pinref part="P+32" gate="VCC" pin="VCC"/>
-<wire x1="-86.36" y1="330.2" x2="-86.36" y2="322.58" width="0.1524" layer="91"/>
-</segment>
-<segment>
-<pinref part="C5" gate="G$1" pin="1"/>
-<wire x1="-66.04" y1="302.26" x2="-66.04" y2="299.72" width="0.1524" layer="91"/>
-<pinref part="P+33" gate="VCC" pin="VCC"/>
-</segment>
-<segment>
 <pinref part="U$5" gate="G$1" pin="VCC"/>
 <wire x1="-83.82" y1="386.08" x2="-83.82" y2="398.78" width="0.1524" layer="91"/>
@@
 </segment>
 <segment>
-<wire x1="0" y1="388.62" x2="-30.48" y2="388.62" width="0.1524" layer="91"/>
 <pinref part="P+23" gate="VCC" pin="VCC"/>
 <wire x1="-30.48" y1="391.16" x2="-30.48" y2="388.62" width="0.1524" layer="91"/>
 <pinref part="SV1" gate="G$1" pin="1"/>
-</segment>
-<segment>
-<wire x1="-20.32" y1="368.3" x2="-20.32" y2="370.84" width="0.1524" layer="91"/>
-<pinref part="P+24" gate="VCC" pin="VCC"/>
-<pinref part="SV1" gate="G$1" pin="17"/>
-<wire x1="0" y1="368.3" x2="-20.32" y2="368.3" width="0.1524" layer="91"/>
+<wire x1="-30.48" y1="388.62" x2="0" y2="388.62" width="0.1524" layer="91"/>
 </segment>
 <segment>
@@
 <junction x="20.32" y="185.42"/>
 <pinref part="+3V13" gate="G$1" pin="+3V3"/>
+<pinref part="V33" gate="G$1" pin="TP"/>
+<junction x="17.78" y="185.42"/>
 </segment>
 <segment>
@@
 </segment>
 </net>
+<net name="V+" class="0">
+<segment>
+<wire x1="-20.32" y1="368.3" x2="-20.32" y2="370.84" width="0.1524" layer="91"/>
+<pinref part="SV1" gate="G$1" pin="17"/>
+<wire x1="0" y1="368.3" x2="-17.78" y2="368.3" width="0.1524" layer="91"/>
+<pinref part="SUPPLY1" gate="1" pin="V+"/>
+<pinref part="VCC" gate="G$1" pin="TP"/>
+<wire x1="-17.78" y1="368.3" x2="-20.32" y2="368.3" width="0.1524" layer="91"/>
+<junction x="-17.78" y="368.3"/>
+</segment>
+<segment>
+<pinref part="R4" gate="G$1" pin="2"/>
+<wire x1="-119.38" y1="330.2" x2="-119.38" y2="322.58" width="0.1524" layer="91"/>
+<pinref part="SUPPLY2" gate="1" pin="V+"/>
+</segment>
+<segment>
+<pinref part="IC2" gate="G$1" pin="VCC"/>
+<wire x1="-96.52" y1="330.2" x2="-96.52" y2="314.96" width="0.1524" layer="91"/>
+<pinref part="SUPPLY3" gate="1" pin="V+"/>
+</segment>
+<segment>
+<pinref part="R5" gate="G$1" pin="2"/>
+<wire x1="-86.36" y1="330.2" x2="-86.36" y2="322.58" width="0.1524" layer="91"/>
+<pinref part="SUPPLY4" gate="1" pin="V+"/>
+</segment>
+<segment>
+<pinref part="C5" gate="G$1" pin="1"/>
+<wire x1="-66.04" y1="302.26" x2="-66.04" y2="299.72" width="0.1524" layer="91"/>
+<pinref part="SUPPLY5" gate="1" pin="V+"/>
+</segment>
+</net>
