File: Eagle/CrackberryPi_1.0.6.2.brd (EAGLE design)
At the start: 85 x 96 mm, 165 parts, among them IC1 REG1117, IC2 24C02CSM, Q1 IRLML5203, Q2 IRLML5203, Q4 IRLML5203, Q5 32.768, T1 BC847, T3 BC847, T4 BC847, X3 C-GRID-03-70543, X5 FH12-50S-0.5SH

Commit message: testing progress
Parts:
- removed C22: 0.1mf, rcl:C0603
- removed C23: 470pf, rcl:C0603
- removed C25: 22uF, rcl:C1206
- removed D4: 1N759, diode:SOD80C
- removed Q2: IRLML5203, transistor-power:MICRO3
- removed R11, R12, R28, R29: 10k, rcl:R0603
- removed SJ1, SJ3, SJ4: (no value), jumper:SJ
- removed T3, T4: BC847, transistor:SOT23
- removed U$10, U$3: MAX2650, max2650:SOT143-W
- removed U$8: MOMSWITCH, momswitch:MOMSWITCH
- added R35, R41: 4k7, rcl:R0603
- added S2: TL49WO, switch:TL4XWO
- added T5, T6, T7: BC847, transistor:SOT23
- C21: value 470pf -> 1uF
- R38: value 30 -> 1.3m
- T2: value (none) -> BC847; device transistor:SOT23-EBC -> transistor:SOT23
- moved C32 77.3 mm to (5.15, 52.0), turned to 0 degrees
- moved C30 76.4 mm to (4.15, 49.6)
- moved R34 76.4 mm to (5.85, 49.7), turned to 270 degrees
- moved U$13 70.8 mm to (8.22, 51.4), turned to 180 degrees
- moved R33 66.8 mm to (11.0, 51.0), turned to 90 degrees
- moved C31 65.3 mm to (12.7, 51.1), turned to 270 degrees
- moved U$7 55.6 mm to (75.8, 29.6), turned to 90 degrees
- moved D2 30.8 mm to (54.8, 91.3), turned to 270 degrees
- moved C15 30.0 mm to (56.0, 86.2), turned to 180 degrees
- moved C9 27.6 mm to (46.1, 51.0)
- moved L2 26.8 mm to (57.6, 91.4), turned to 270 degrees
- moved U$9 22.9 mm to (83.8, 74.0), turned to 270 degrees
- moved T2 22.3 mm to (60.7, 86.8)
- moved C12 20.5 mm to (61.1, 92.7), turned to 0 degrees
- moved C5 17.8 mm to (64.0, 84.5), turned to 270 degrees
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Connections:
- removed net GPIO16: U$11.P$36
- removed net GPIO20: U$11.P$38
- removed net IN_1: C21.2, U$3.1
- removed net N$13: Q2.1, R11.1, T3.3
- removed net N$17: R12.1, T3.1, U$8.2
- removed net N$22: R29.1, T4.3, U$8.1
- removed net N$24: C25.2, R28.1, T4.1
- removed net OUT1_IN2: U$10.1, U$3.3
- removed net OUT2: C23.2, U$10.3
- removed net VBAT_+: BATTERY.1, Q2.2, R11.2, R29.2, SJ3.2
- new net GPIO27: U$11.P$13
- new net N$28: C21.1, R35.1, T5.3, T7.2
- new net N$32: C21.2, R38.1, T6.1
- new net RANDOM_POWER: R38.2, R41.2, U$11.P$40
- net +15V: now also R35.2; no longer D4.C
- net +3V3: now also C30.1, C31.1, R33.2, R34.2, U$13.1, U$13.8; no longer U$7.38, U$7.39
- net +5V: now also T2.2; no longer C22.2, SJ1.1, SJ1.2, SJ4.1, T2.E, U$10.4, U$3.4
- net BAT: now also BATTERY.1; no longer Q2.3, R12.2, R28.2, SJ3.1
- net DISPLAY_RESET: now also U$11.P$29; no longer U$11.P$33
- net GND: now also T5.2, T6.2; no longer C22.1, C25.1, R38.1, T3.2, T4.2, U$10.2, U$3.2
- net HVOUT: now also T2.3; no longer T2.C
- net HVPR: now also T2.1; no longer T2.B
- net IN: no longer SJ4.2
- net INT_KB: now also U$11.P$38; no longer U$11.P$40
- net IR_TX: now also U$11.P$35; no longer U$11.P$13
- net N$1: now also Q3.4; no longer Q3.1
- net N$16: now also T5.1, T7.1; no longer C21.1, D4.A, R38.2
- net N$2: now also Q3.1; no longer Q3.4
- net PWM: now also U$11.P$33; no longer U$11.P$29
- net RANDOM: now also R41.1, T6.3; no longer C23.1
- net STEPUP_ENABLE: now also U$11.P$36; no longer U$11.P$35
- net V+: no longer C30.1, C31.1, R33.2, R34.2, U$13.1, U$13.8
- net VCC: now also U$7.38, U$7.39
Routing:
- net SDA_3V3: track 141.4 -> 68.1 mm, vias 7 -> 6
- net SCL_3V3: track 142.3 -> 79.9 mm, vias 3 -> 5
- net +5V: track 277.8 -> 221.1 mm, vias 9 -> 6
- net ROW10: track 86.3 -> 34.0 mm
- net INT_KB: track 7.69 -> 55.5 mm, vias 0 -> 1
- net ACC_INT2: track 46.9 -> 0.00 mm, vias 1 -> 0
- net ROW9: track 87.8 -> 42.3 mm
- net ROW0: track 64.8 -> 105.2 mm, vias 2 -> 1
- net ACC_INT1: track 40.0 -> 0.00 mm, vias 1 -> 0
- net ROW1: track 50.1 -> 88.3 mm, vias 2 -> 1
- net +3V3: track 128.0 -> 91.0 mm, vias 4 -> 2
- net ROW2: track 54.1 -> 89.7 mm, vias 2 -> 1
- net BAT: track 42.6 -> 8.46 mm, vias 4 -> 0
- net ROW3: track 50.4 -> 82.9 mm, vias 2 -> 1
- net V+: track 57.0 -> 28.5 mm, vias 2 -> 0
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- added copper zone on layer 16, net IN
- removed copper zone on layer 16, net HVPR
- removed copper zone on layer 16, net VBAT_+

Commit message: lots of updates
Parts:
- removed LED1: (no value), led:CHIP-LED0603
- removed R30: 30, rcl:R0603
- removed S2: TL49WO, switch:TL4XWO
- removed SJ2: (no value), jumper:SJ
- added C22: 100nF, rcl:C0603
- added C23: 1mf, rcl:C0603
- added SJ1: (no value), jumper:SJ
- added U$3: RESETMONITOR, MAX803:SOT23
- moved C13 47.0 mm to (72.6, 80.7), turned to 180 degrees
- moved BATTERY 42.8 mm to (83.8, 40.5), flipped to the bottom, turned to 180 degrees
- moved C30 38.7 mm to (33.3, 75.1), turned to 270 degrees
- moved IC1 38.1 mm to (67.5, 75.9), turned to 180 degrees
- moved C14 36.3 mm to (65.7, 81.8), turned to 270 degrees
- moved R34 36.1 mm to (31.6, 75.0), turned to 90 degrees
- moved R33 32.4 mm to (29.5, 77.5), turned to 0 degrees
- moved U$13 31.3 mm to (29.1, 74.7), turned to 90 degrees
- moved C32 30.4 mm to (26.6, 73.5), turned to 270 degrees
- moved C31 29.3 mm to (26.6, 76.8)
- moved C1 24.0 mm to (64.1, 81.8), turned to 270 degrees
- moved U$9 23.0 mm to (76.5, 95.8), turned to 180 degrees
- moved C6 17.2 mm to (22.5, 72.0), turned to 180 degrees
- moved C5 14.8 mm to (78.0, 89.4), turned to 180 degrees
- moved L1 13.9 mm to (25.0, 69.1), turned to 270 degrees
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Connections:
- removed net EMITTER: T1.2
- removed net N$11: LED1.C, R30.2
- removed net STEPUP_ENABLE: U$11.P$36, U$2.1
- new net GPIO16: U$11.P$36
- new net GPIO5: U$11.P$29
- net +3V3: now also C22.1, U$3.3
- net +5V: now also C23.1, SJ1.2; no longer LED1.A, SJ2.1, SJ2.2
- net DISPLAY_RESET: now also U$3.2; no longer U$11.P$29
- net GND: now also C22.2, C23.2, T1.2, U$3.1; no longer R30.1
- net IN: now also SJ1.1
- net RANDOM_POWER: now also U$2.1
Routing:
- net +3V3: track 91.0 -> 180.5 mm
- net SCL_3V3: track 79.9 -> 150.1 mm, vias 5 -> 6
- net SDA_3V3: track 68.1 -> 130.1 mm
- net ACC_INT1: track 0.00 -> 56.2 mm, vias 0 -> 1
- net BAT: track 8.46 -> 61.1 mm, vias 0 -> 3
- net ACC_INT2: track 0.00 -> 52.6 mm, vias 0 -> 1
- net RANDOM_POWER: track 8.30 -> 49.4 mm, vias 0 -> 1
- net DISPLAY_RESET: track 40.2 -> 7.11 mm, vias 1 -> 0
- net STEPUP_ENABLE: track 25.1 -> 0.00 mm, vias 1 -> 0
- net HVPR: track 4.60 -> 24.6 mm, vias 0 -> 2
- net +5V: track 221.1 -> 201.7 mm, vias 6 -> 7
- net GND: track 137.3 -> 128.9 mm, vias 25 -> 88
- net N$7: track 15.3 -> 8.74 mm
- net +15V: track 7.84 -> 14.2 mm
- net VBAT+: track 12.3 -> 6.62 mm
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- removed copper zone on layer 16, net +3V3
Other:
- board size 85 x 96 mm -> 87 x 98 mm
