File: Eagle/CrackberryPi_1.0.6.2.sch (EAGLE design)
At the start: 149 parts, among them IC1 REG1117, IC2 24C02CSM, Q1 IRLML5203, Q2 32.768, T1 BC847, X1 53261-02, X3 C-GRID-03-70543, X5 FH12-50S-0.5SH

Commit message: lots of pcb progress and iterations
Parts:
- removed SV1: (no value), con-lsta:FE20-2
- removed SV3: (no value), con-lsta:FE09-2
- removed TP1, TP2: TPTP20SQ, testpad:TPTP20SQ
- removed X1: 53261-02, con-molex:53261-02
- added BATTERY: 22-27-2021-02, con-molex:22-27-2021-02
- added C29: 22nF, rcl:C-EUC0603
- added C30, C32: 0.1mf, rcl:C-EUC0603
- added C31: 1mf, rcl:C-EUC0603
- added Q4: IRLML5203, transistor-power:IRLML5203
- added Q5: 32.768, crystal:CRYSTALMM20SS
- added R30: 30, rcl:R-EU_R0603
- added R31, R32: 10k, rcl:R-EU_R0603
- added R33, R34: 3.9K, rcl:R-EU_R0603
- added SJ1, SJ3, SJ4: (no value), jumper:SJ
- added T2: (no value), transistor:-NPN-SOT23-EBC
- added T3, T4: BC847, transistor:BC847
- added U$11: HEADER, 20x2_cirqoid:HEADER
- added U$12: SI4713, Si4713:SI4713
- added U$13: ACCELLEROMETER, MMA8653:ACCELLEROMETER
- C1, C5: value (none) -> 4.7mF
- C10: value 0.047mF -> .1mF
- C11: value 4.7mF -> 270pF
- C12: value 4.7mF -> 0.47mF
- C15: value 10mF -> 22uF; device rcl:C-EUC0603 -> rcl:C-EUC1206
- C25: value 0.47uF -> 22uF; device rcl:C-EUC0603 -> rcl:C-EUC1206
- C27: value 10uF -> 0.47uF
- C28: value 22nF -> 10uF
- D2: value BB141 -> (none); device diode:BB141 -> diode:DIODE-SOD123
- L1: device rcl:R-EU_R1206W -> rcl:R-EU_R0805
- L2: value 8.2mH -> 6.8uH; device rcl:R-EU_R1206W -> rcl:R-EU_R2010
- LED1: device led:LEDSML0603 -> led:LEDCHIP-LED0603
- Q2: value 32.768 -> IRLML5203; device crystal:CRYSTALMM20SS -> transistor-power:IRLML5203
- R10: value 10k -> 40.2k
- R12: value 30 -> 10k
- R27: value 10k -> 1k
- R7: value THERMISTOR-2,5 -> 59k; device varistor:THERMISTOR-2,5 -> rcl:R-EU_R0603
- R8: value 317 -> 2.1k
- R9: value 10k -> 71.5k
- U$1: value BQ24297 -> LTC4090; device BQ24297:BQ24297 -> LTC4090:LTC4090
- U$8: value SI4713 -> MOMSWITCH; device Si4713:SI4713 -> momswitch:MOMSWITCH
- renumbered + to 12, - to 11, 0 to 10
Connections:
- removed net AVALANCHE_ENABLE: SV1.40
- removed net GPIO18: SV1.12
- removed net GPIO19: SV1.35
- removed net GPIO23: SV1.16, SV3.9
- removed net GPIO25: SV1.22, SV3.12
- removed net GPIO27: SV1.13, SV3.8
- removed net GPIO5: SV1.29
- removed net INT: SV1.7, SV3.2, U$1.INT, U$5.INT, U$6.INT, U$7.INT
- removed net VBUS: C16.1, U$1.VBUS, U$9.1_+5V
- new net ACC_INT1: U$11.P$12, U$13.INT1
- new net ACC_INT2: U$11.P$16, U$13.INT2
- new net BAT: Q2.D, Q4.D, R12.2, R28.2, SJ3.1, U$1.BAT
- new net BOOST: C12.1, U$1.BOOST
- new net D/C: U$11.P$22, X5-37.1
- new net GPIO12: U$11.P$32
- new net GPIO16: U$11.P$36
- new net GPIO20: U$11.P$38
- new net HVOUT: C15.2, L2.2, T2.C, U$1.HVOUT
- new net HVPR: R27.1, T2.B, U$1.HVPR
- new net IN: C17.1, C5.1, SJ4.2, U$1.HPWR, U$1.IN, U$9.1_+5V
- new net INT_KB: U$11.P$40, U$7.INT
- new net INT_RTC: U$11.P$7, U$5.INT
- new net INT_TOUCH: U$11.P$31, U$6.INT
- new net N$27: R26.2, U$1.NTC
- new net N$29: R32.2, U$12.SEN
- new net N$31: C32.1, U$13.BYP
- new net N$33: Q4.G, U$1.GATE
- new net SW: C12.2, D2.C, L2.1, U$1.SW
- new net V+: C30.1, C31.1, IC2.VCC, R33.2, R34.2, R4.2, R5.2, U$11.P$17, U$13.VDD, U$13.VDDIO, U$5.VCC
- new net VBAT_+: BATTERY-1.S, Q2.S, R11.2, R29.2, SJ3.2
- net +3V3: now also C1.1, C29.1, R25.1, R31.1, R32.1, U$12.VDD, U$12.VIO, U$7.VCC; no longer C27.1, R10.1, R11.1, R28.1, R29.1, R39.2, R9.1, SV3.17, SV3.7, U$1.SYS, U$8.VDD, U$8.VIO, X5-37.1
- net +5V: now also C16.1, LED1.A, Q4.S, R27.2, R39.2, SJ1.1, SJ1.2, SJ4.1, T2.E, U$1.OUT, U$11.P$2, U$11.P$4; no longer C11.1, L2.2, R12.1, SV1.2, SV1.4, SV3.18
- net AUDIO_L: now also C26.1; no longer C25.1
- net AUDIO_R: now also C27.1; no longer C26.1
- net CE0: now also U$11.P$24; no longer SV1.24
- net CE1: now also U$11.P$26; no longer SV1.26
- net D+: no longer U$1.D+/PSEL
- net D-: no longer U$1.D-/PG
- net DISPLAY_RESET: now also U$11.P$33; no longer SV1.33
- net FM_RST: now also R31.2, U$12.RST; no longer D2.C, SV1.37
- net GND: now also BATTERY-2.S, C10.1, C11.1, C15.1, C25.1, C29.2, C30.2, C31.2, C32.2, D2.A, R10.2, R30.1, R9.2, T3.E, T4.E, U$1.GND, U$1.SUSP, U$1.SYNC, U$11.P$14, U$11.P$20, U$11.P$25, U$11.P$30, U$11.P$34, U$11.P$39, U$11.P$6, U$11.P$9, U$12.DFN, U$12.DIN, U$12.GND, U$12.RFGND, U$13.GND; no longer C11.2, C12.2, C15.2, C27.2, R25.1, R26.2, R27.1, R7.2, SV1.14, SV1.20, SV1.25, SV1.30, SV1.34, SV1.39, SV1.6, SV1.9, SV3.15, SV3.5, TP2.TP, U$1.PGND, U$8.DFN, U$8.DIN, U$8.GND, U$8.RFGND, X1-2.S
- net GPIO22: now also U$11.P$15; no longer SV1.15, SV3.10
- net GPIO24: now also U$11.P$18; no longer SV1.18, SV3.11
- net GPO1: now also U$12.GPO1; no longer U$8.GPO1
- net GPO2: now also U$12.GPO2; no longer U$8.GPO2
- net ID_SC: now also U$11.P$28; no longer SV1.28
- net ID_SD: now also U$11.P$27; no longer SV1.27
- net IR_RX: now also U$11.P$11; no longer SV1.36
- net IR_TX: now also U$11.P$13; no longer SV1.38
- net MISO: now also U$11.P$21; no longer SV1.21, SV3.13
- net MOSI: now also U$11.P$19; no longer SV1.19, SV3.14
- net N$1: now also Q3.1, U$5.X2; no longer C10.1, L2.1, U$1.SW
- net N$11: now also LED1.C, R30.2; no longer Q3.1, U$5.X1
- net N$13: now also Q2.G, R11.1, T3.C; no longer Q3.2, U$5.X2
- net N$15: now also C8.1, Q5.1, U$12.RCLK; no longer R27.2, U$1.CE
- net N$17: now also R12.1, T3.B, U$8.2; no longer R28.2, U$1.OTG
- net N$19: now also Q5.2, U$12.GPO3; no longer Q2.2, U$8.GPO3
- net N$2: now also Q3.2, U$5.X1; no longer C10.2, U$1.BTST
- net N$21: now also R26.1, U$1.VNTC; no longer C8.1, Q2.1, U$8.RCLK
- net N$22: now also R29.1, T4.C, U$8.1; no longer C25.2, U$8.LIN
- net N$23: now also U$12.LIN; no longer U$8.RIN
- net N$24: now also C25.2, R28.1, T4.B; no longer D2.A, R11.2, U$8.RST
- net N$25: now also C27.2, U$12.RIN; no longer ANTENNA.MP, L3.2, U$8.TX0
- net N$26: now also ANTENNA.MP, L3.2, U$12.TX0; no longer R29.2, U$8.SEN
- net N$3: now also R9.1, U$1.PROG; no longer C15.1, TP1.TP, U$1.BAT, X1-1.S
- net N$4: now also R10.1, U$1.RT; no longer LED1.A, R12.2
- net N$5: now also R8.1, U$1.CLPROG; no longer C12.1, U$1.REGN
- net N$6: now also U$1.VC; no longer R26.1, U$1.TS
- net N$7: now also C10.2, U$1.TIMER; no longer R8.1, U$1.ILIM
- net N$8: now also C11.2, R7.2; no longer C17.1, U$1.PMD
- net N$9: now also U$1.HVEN, U$1.HVIN; no longer LED1.C, U$1.STAT
- net PWM: now also U$11.P$29; no longer SV1.11
- net RANDOM: now also U$11.P$37; no longer SV1.32
- net SCK: now also U$11.P$23; no longer SV1.23, SV3.16
- net SCL_3V3: now also R34.1, U$11.P$5, U$12.SCLK, U$13.SCL; no longer R10.2, SV1.5, SV3.6, U$1.SCL, U$8.SCLK
- net SDA_3V3: now also R33.1, U$11.P$3, U$12.SDIO, U$13.SDA; no longer R9.2, SV1.3, SV3.4, U$1.SDA, U$8.SDIO
- net STEPUP_ENABLE: now also U$11.P$35; no longer SV1.31
- net UART_RX: now also U$11.P$10; no longer SV1.10, SV3.3
- net UART_TX: now also U$11.P$8; no longer SV1.8, SV3.1
- net VCC: now also U$11.P$1; no longer C1.1, C5.1, IC2.VCC, R4.2, R5.2, SV1.1, SV1.17, U$5.VCC, U$7.VCC
Other:
- moved on the sheet: ANTENNA, AUDIO_L, AUDIO_R, C1, C10, C11, C12, C13, C14, C15, C16, C17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

Commit message: testing progress
Parts:
- removed C22: 0.1mf, rcl:C-EUC0603
- removed C23: 470pf, rcl:C-EUC0603
- removed C25: 22uF, rcl:C-EUC1206
- removed D4: 1N759, diode:ZENER-DIODESOD80C
- removed Q2: IRLML5203, transistor-power:IRLML5203
- removed R11, R12, R28, R29: 10k, rcl:R-EU_R0603
- removed SJ1, SJ3, SJ4: (no value), jumper:SJ
- removed T3, T4: BC847, transistor:BC847
- removed U$10, U$3: MAX2650, max2650:MAX2650
- removed U$8: MOMSWITCH, momswitch:MOMSWITCH
- added R35, R41: 4k7, rcl:R-EU_R0603
- added S2: TL49WO, switch:TL49WO
- added T5, T6, T7: BC847, transistor:BC847
- C21: value 470pf -> 1uF
- R38: value 30 -> 1.3m
- T2: value (none) -> BC847; device transistor:-NPN-SOT23-EBC -> transistor:BC847
Connections:
- removed net GPIO16: U$11.P$36
- removed net GPIO20: U$11.P$38
- removed net IN_1: C21.2, U$3.IN
- removed net N$13: Q2.G, R11.1, T3.C
- removed net N$17: R12.1, T3.B, U$8.2
- removed net N$22: R29.1, T4.C, U$8.1
- removed net N$24: C25.2, R28.1, T4.B
- removed net OUT1_IN2: U$10.IN, U$3.OUT
- removed net OUT2: C23.2, U$10.OUT
- removed net VBAT_+: BATTERY-1.S, Q2.S, R11.2, R29.2, SJ3.2
- new net GPIO27: U$11.P$13
- new net N$28: C21.1, R35.1, T5.C, T7.E
- new net N$32: C21.2, R38.1, T6.B
- new net RANDOM_POWER: R38.2, R41.2, U$11.P$40
- net +15V: now also R35.2; no longer D4.C
- net +3V3: now also C30.1, C31.1, R33.2, R34.2, U$13.VDD, U$13.VDDIO; no longer U$7.VCC
- net +5V: no longer C22.2, SJ1.1, SJ1.2, SJ4.1, U$10.VCC, U$3.VCC
- net BAT: now also BATTERY-1.S; no longer Q2.D, R12.2, R28.2, SJ3.1
- net DISPLAY_RESET: now also U$11.P$29; no longer U$11.P$33
- net GND: now also T5.E, T6.E; no longer C22.1, C25.1, R38.1, T3.E, T4.E, U$10.GND, U$3.GND
- net IN: no longer SJ4.2
- net INT_KB: now also U$11.P$38; no longer U$11.P$40
- net IR_TX: now also U$11.P$35; no longer U$11.P$13
- net N$1: now also Q3.2; no longer Q3.1
- net N$16: now also T5.B, T7.B; no longer C21.1, D4.A, R38.2
- net N$2: now also Q3.1; no longer Q3.2
- net PWM: now also U$11.P$33; no longer U$11.P$29
- net RANDOM: now also R41.1, T6.C; no longer C23.1
- net STEPUP_ENABLE: now also U$11.P$36; no longer U$11.P$35
- net V+: no longer C30.1, C31.1, R33.2, R34.2, U$13.VDD, U$13.VDDIO
- net VCC: now also U$7.VCC
Other:
- moved on the sheet: BATTERY-1, BATTERY-2, C19, C21, Q3, R38

Commit message: lots of updates
Parts:
- removed LED1: (no value), led:LEDCHIP-LED0603
- removed R30: 30, rcl:R-EU_R0603
- removed S2: TL49WO, switch:TL49WO
- removed SJ2: (no value), jumper:SJ
- added C22: 100nF, rcl:C-EUC0603
- added C23: 1mf, rcl:C-EUC0603
- added SJ1: (no value), jumper:SJ
- added U$3: RESETMONITOR, MAX803:RESETMONITOR
Connections:
- removed net EMITTER: T1.E
- removed net N$11: LED1.C, R30.2
- removed net STEPUP_ENABLE: U$11.P$36, U$2.CE
- new net GPIO16: U$11.P$36
- new net GPIO5: U$11.P$29
- net +3V3: now also C22.1, U$3.VCC
- net +5V: now also C23.1, SJ1.2; no longer LED1.A, SJ2.1, SJ2.2
- net DISPLAY_RESET: now also U$3.RESET; no longer U$11.P$29
- net GND: now also C22.2, C23.2, T1.E, U$3.GND; no longer R30.1
- net IN: now also SJ1.1
- net RANDOM_POWER: now also U$2.CE
Other:
- moved on the sheet: C13, C14, IC1
